File: packages/connectors/layouts/addressable_led_connector/addressable_led_connector.kicad_pcb (KiCad board)
At the start: 2 copper layers, 1 part

Commit message: Update build script and regenerate outputs
Connections:
- U1 pad 3: line-1 -> line
- U1 pad 4: line -> line-1
Changed lines of the file:
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@@
     )
     (net 0 "")
-    (net 1 "line-1")
+    (net 1 "line")
     (net 2 "gnd")
-    (net 3 "line")
+    (net 3 "line-1")
     (net 4 "hv")
     (footprint "atopile:CONN-TH_4P-XT30PW-M-e6a65c"
@@
             (drill 0.9144)
             (layers "*.Cu" "*.Mask")
-            (net 1 "line-1")
+            (net 1 "line")
         )
         (pad "4" thru_hole circle
@@
             (drill 0.9144)
             (layers "*.Cu" "*.Mask")
-            (net 3 "line")
+            (net 3 "line-1")
         )
     )
