File: packages/logic/layouts/aip74lvc1t45/aip74lvc1t45.kicad_pcb (KiCad board)
At the start: 2 copper layers, 3 parts

Commit message: Rebuild modules frozen (#12)
* Rebuild logic package

* Add updated docs for logic package

* Rebuild relays package

* Rebuild usb package

* Rebuild switches package

* Rebuild rs485 package

* Add option to specify package to doc generator

* Add updated docs for rs485 package

* Update main README
Connections:
- C1 pad 1: hv-1 -> hv
- C2 pad 1: hv -> hv-1
- U1 pad 1: hv-1 -> hv
- U1 pad 3: buffer-line-2 -> buffer-line-1
- U1 pad 5: buffer-line-1 -> buffer-line-2
- U1 pad 6: hv -> hv-1
Changed lines of the file:
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@@
     )
     (net 0 "")
-    (net 1 "hv")
-    (net 2 "hv-1")
+    (net 1 "hv-1")
+    (net 2 "hv")
     (net 3 "gnd")
-    (net 4 "buffer-line-1")
+    (net 4 "buffer-line-2")
     (net 5 "buffer-line")
-    (net 6 "buffer-line-2")
+    (net 6 "buffer-line-1")
     (footprint "atopile:SOT-23-6_L2.9-W1.6-P0.95-LS2.8-BL-d2c740"
         (layer "F.Cu")
@@
             (size 0.53 1.07)
             (layers "F.Cu" "F.Mask" "F.Paste")
-            (net 2 "hv-1")
+            (net 2 "hv")
         )
         (pad "2" smd rect
@@
             (size 0.53 1.07)
             (layers "F.Cu" "F.Mask" "F.Paste")
-            (net 6 "buffer-line-2")
+            (net 6 "buffer-line-1")
         )
         (pad "4" smd rect
@@
             (size 0.53 1.07)
             (layers "F.Cu" "F.Mask" "F.Paste")
-            (net 4 "buffer-line-1")
+            (net 4 "buffer-line-2")
         )
         (pad "6" smd rect
@@
             (size 0.53 1.07)
             (layers "F.Cu" "F.Mask" "F.Paste")
-            (net 1 "hv")
+            (net 1 "hv-1")
         )
         (embedded_fonts no)
@@
             (size 0.79 0.54)
             (layers "F.Cu" "F.Mask" "F.Paste")
-            (net 1 "hv")
+            (net 1 "hv-1")
         )
         (pad "2" smd rect
@@
             (size 0.79 0.54)
             (layers "F.Cu" "F.Mask" "F.Paste")
-            (net 2 "hv-1")
+            (net 2 "hv")
         )
         (pad "2" smd rect
