File: packages/logic/layouts/iso1540/iso1540.kicad_pcb (KiCad board)
At the start: 2 copper layers, 3 parts

Commit message: Rebuild modules frozen (#12)
* Rebuild logic package

* Add updated docs for logic package

* Rebuild relays package

* Rebuild usb package

* Rebuild switches package

* Rebuild rs485 package

* Add option to specify package to doc generator

* Add updated docs for rs485 package

* Update main README
Connections:
- C1 pad 1: hv -> hv-1
- C2 pad 1: hv-1 -> hv
- U1 pad 1: hv-1 -> hv
- U1 pad 2: line-2 -> line-3
- U1 pad 3: line-1 -> line
- U1 pad 6: line -> line-2
- U1 pad 7: line-3 -> line-1
- U1 pad 8: hv -> hv-1
Changed lines of the file:
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@@
     )
     (net 0 "")
-    (net 1 "line")
-    (net 2 "line-3")
-    (net 3 "line-1")
-    (net 4 "line-2")
+    (net 1 "line-2")
+    (net 2 "line-1")
+    (net 3 "line")
+    (net 4 "line-3")
     (net 5 "gnd")
-    (net 6 "hv-1")
-    (net 7 "hv")
+    (net 6 "hv")
+    (net 7 "hv-1")
     (net 8 "gnd-1")
     (footprint "atopile:SOIC-8_L4.9-W3.9-P1.27-LS6.0-BL-6ccfeb"
@@
             (size 0.59 2.05)
             (layers "F.Cu" "F.Mask" "F.Paste")
-            (net 6 "hv-1")
+            (net 6 "hv")
         )
         (pad "2" smd oval
@@
             (size 0.59 2.05)
             (layers "F.Cu" "F.Mask" "F.Paste")
-            (net 4 "line-2")
+            (net 4 "line-3")
         )
         (pad "3" smd oval
@@
             (size 0.59 2.05)
             (layers "F.Cu" "F.Mask" "F.Paste")
-            (net 3 "line-1")
+            (net 3 "line")
         )
         (pad "4" smd oval
@@
             (size 0.59 2.05)
             (layers "F.Cu" "F.Mask" "F.Paste")
-            (net 1 "line")
+            (net 1 "line-2")
         )
         (pad "7" smd oval
@@
             (size 0.59 2.05)
             (layers "F.Cu" "F.Mask" "F.Paste")
-            (net 2 "line-3")
+            (net 2 "line-1")
         )
         (pad "8" smd oval
@@
             (size 0.59 2.05)
             (layers "F.Cu" "F.Mask" "F.Paste")
-            (net 7 "hv")
+            (net 7 "hv-1")
         )
         (embedded_fonts no)
@@
             (size 0.79 0.54)
             (layers "F.Cu" "F.Mask" "F.Paste")
-            (net 7 "hv")
+            (net 7 "hv-1")
         )
         (pad "2" smd rect
@@
             (size 0.79 0.54)
             (layers "F.Cu" "F.Mask" "F.Paste")
-            (net 6 "hv-1")
+            (net 6 "hv")
         )
         (pad "2" smd rect
