File: packages/logos/layouts/faebryk_8x9mm/faebryk_8x9mm.kicad_pcb (KiCad board)
At the start: 2 copper layers, 1 part

Commit message: Update logos package
Parts:
- LOGO1: footprint atopile:faebrykLogo_8x9mm-fe4042 -> lib:faebrykLogo_8x9mm
Changed lines of the file:
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@@
     )
     (net 0 "")
-    (footprint "atopile:faebrykLogo_8x9mm-fe4042"
+    (footprint "lib:faebrykLogo_8x9mm"
         (layer "F.Cu")
         (at 0 0 0)
