File: packages/esp32s3/layouts/esp32_s3_wroom_reference_design/esp32_s3_wroom_reference_design.kicad_pcb (KiCad board)
At the start: 2 copper layers, 7 parts

Commit message: Work around bad atopile net handling
Mannually remove net number gap in pcb file and rebuild
Connections:
- U2 pad 10: line-28 -> line-2
- U2 pad 11: line-29 -> line-20
- U2 pad 12: line-9 -> line-18
- U2 pad 13: line-26 -> line-15
- U2 pad 14: line-15 -> line-27
- U2 pad 15: line-21 -> line-7
- U2 pad 16: line -> line-24
- U2 pad 17: line-24 -> line-19
- U2 pad 18: line-33 -> line-1
- U2 pad 19: line-6 -> line
- U2 pad 20: line-13 -> line-11
- U2 pad 21: line-1 -> line-16
- U2 pad 22: line-23 -> line-17
- U2 pad 23: line-25 -> line-14
- U2 pad 24: line-32 -> line-12
- U2 pad 25: line-11 -> line-30
- U2 pad 26: line-3 -> line-9
- U2 pad 28: line-2 -> line-22
- U2 pad 29: line-34 -> line-26
- U2 pad 30: line-10 -> line-28
- U2 pad 31: line-22 -> line-34
- U2 pad 32: line-7 -> line-4
- U2 pad 33: line-14 -> line-5
- U2 pad 34: line-8 -> line-10
- U2 pad 35: line-27 -> line-32
- U2 pad 36: line-17 -> line-21
- U2 pad 37: line-16 -> line-8
- U2 pad 38: line-5 -> line-3
- U2 pad 39: line-30 -> line-23
- U2 pad 4: line-31 -> line-13
- U2 pad 5: line-19 -> line-31
- U2 pad 6: line-20 -> line-25
- U2 pad 7: line-18 -> line-6
- U2 pad 8: line-12 -> line-29
- U2 pad 9: line-4 -> line-33
Changed lines of the file:
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@@
     )
     (net 0 "")
-    (net 1 "line-26")
-    (net 2 "line-4")
-    (net 3 "line-1")
-    (net 4 "line-13")
-    (net 5 "line-9")
-    (net 6 "line-18")
-    (net 7 "line-7")
-    (net 8 "line-29")
-    (net 9 "line-22")
-    (net 10 "line-8")
-    (net 11 "line-2")
-    (net 12 "line-28")
-    (net 13 "line-14")
+    (net 1 "line-15")
+    (net 2 "line-33")
+    (net 3 "line-16")
+    (net 4 "line-11")
+    (net 5 "line-18")
+    (net 6 "line-6")
+    (net 7 "line-4")
+    (net 8 "line-20")
+    (net 9 "line-34")
+    (net 10 "line-10")
+    (net 11 "line-22")
+    (net 12 "line-2")
+    (net 13 "line-5")
     (net 14 "out")
-    (net 15 "line-30")
-    (net 16 "line-16")
-    (net 17 "line-31")
-    (net 18 "line-34")
-    (net 19 "line-3")
-    (net 20 "line-15")
-    (net 21 "line-25")
-    (net 22 "line-10")
-    (net 23 "line-6")
-    (net 24 "line-17")
-    (net 25 "line-27")
-    (net 26 "line-11")
+    (net 15 "line-23")
+    (net 16 "line-8")
+    (net 17 "line-13")
+    (net 18 "line-26")
+    (net 19 "line-9")
+    (net 20 "line-27")
+    (net 21 "line-14")
+    (net 22 "line-28")
+    (net 23 "line")
+    (net 24 "line-21")
+    (net 25 "line-32")
+    (net 26 "line-30")
     (net 27 "hv")
-    (net 28 "line-32")
-    (net 29 "line-33")
-    (net 30 "line-12")
-    (net 31 "line-21")
-    (net 32 "line-5")
-    (net 33 "line-24")
-    (net 34 "line")
-    (net 35 "line-19")
-    (net 36 "line-20")
-    (net 37 "line-23")
+    (net 28 "line-12")
+    (net 29 "line-1")
+    (net 30 "line-29")
+    (net 31 "line-7")
+    (net 32 "line-3")
+    (net 33 "line-19")
+    (net 34 "line-24")
+    (net 35 "line-31")
+    (net 36 "line-25")
+    (net 37 "line-17")
     (net 38 "gnd")
-    (net 41 "in")
+    (net 39 "in")
     (footprint "atopile:R0402-56259e"
         (layer "F.Cu")
@@
             (size 0.57 0.54)
             (layers "F.Cu" "F.Mask" "F.Paste")
-            (net 41 "in")
+            (net 39 "in")
         )
         (embedded_fonts no)
@@
             (size 1.5 0.9)
             (layers "F.Cu" "F.Mask" "F.Paste")
-            (net 41 "in")
+            (net 39 "in")
         )
         (pad "4" smd rect
@@
             (size 1.5 0.9)
             (layers "F.Cu" "F.Mask" "F.Paste")
-            (net 17 "line-31")
+            (net 17 "line-13")
         )
         (pad "5" smd rect
@@
             (size 1.5 0.9)
             (layers "F.Cu" "F.Mask" "F.Paste")
-            (net 35 "line-19")
+            (net 35 "line-31")
         )
         (pad "6" smd rect
@@
             (size 1.5 0.9)
             (layers "F.Cu" "F.Mask" "F.Paste")
-            (net 36 "line-20")
+            (net 36 "line-25")
         )
         (pad "7" smd rect
@@
             (size 1.5 0.9)
             (layers "F.Cu" "F.Mask" "F.Paste")
-            (net 6 "line-18")
+            (net 6 "line-6")
         )
         (pad "8" smd rect
@@
             (size 1.5 0.9)
             (layers "F.Cu" "F.Mask" "F.Paste")
-            (net 30 "line-12")
+            (net 30 "line-29")
         )
         (pad "9" smd rect
@@
             (size 1.5 0.9)
             (layers "F.Cu" "F.Mask" "F.Paste")
-            (net 2 "line-4")
+            (net 2 "line-33")
         )
         (pad "10" smd rect
@@
             (size 1.5 0.9)
             (layers "F.Cu" "F.Mask" "F.Paste")
-            (net 12 "line-28")
+            (net 12 "line-2")
         )
         (pad "11" smd rect
@@
             (size 1.5 0.9)
             (layers "F.Cu" "F.Mask" "F.Paste")
-            (net 8 "line-29")
+            (net 8 "line-20")
         )
         (pad "12" smd rect
@@
             (size 1.5 0.9)
             (layers "F.Cu" "F.Mask" "F.Paste")
-            (net 5 "line-9")
+            (net 5 "line-18")
         )
         (pad "13" smd rect
@@
             (size 1.5 0.9)
             (layers "F.Cu" "F.Mask" "F.Paste")
-            (net 1 "line-26")
+            (net 1 "line-15")
         )
         (pad "14" smd rect
@@
             (size 1.5 0.9)
             (layers "F.Cu" "F.Mask" "F.Paste")
-            (net 20 "line-15")
+            (net 20 "line-27")
         )
         (pad "15" smd rect
@@
             (size 1.5 0.9)
             (layers "F.Cu" "F.Mask" "F.Paste")
-            (net 31 "line-21")
+            (net 31 "line-7")
         )
         (pad "16" smd rect
@@
             (size 1.5 0.9)
             (layers "F.Cu" "F.Mask" "F.Paste")
-            (net 34 "line")
+            (net 34 "line-24")
         )
         (pad "17" smd rect
@@
             (size 1.5 0.9)
             (layers "F.Cu" "F.Mask" "F.Paste")
-            (net 33 "line-24")
+            (net 33 "line-19")
         )
         (pad "18" smd rect
@@
             (size 1.5 0.9)
             (layers "F.Cu" "F.Mask" "F.Paste")
-            (net 29 "line-33")
+            (net 29 "line-1")
         )
         (pad "19" smd rect
@@
             (size 1.5 0.9)
             (layers "F.Cu" "F.Mask" "F.Paste")
-            (net 23 "line-6")
+            (net 23 "line")
         )
         (pad "20" smd rect
@@
             (size 1.5 0.9)
             (layers "F.Cu" "F.Mask" "F.Paste")
-            (net 4 "line-13")
+            (net 4 "line-11")
         )
         (pad "21" smd rect
@@
             (size 1.5 0.9)
             (layers "F.Cu" "F.Mask" "F.Paste")
-            (net 3 "line-1")
+            (net 3 "line-16")
         )
         (pad "22" smd rect
@@
             (size 1.5 0.9)
             (layers "F.Cu" "F.Mask" "F.Paste")
-            (net 37 "line-23")
+            (net 37 "line-17")
         )
         (pad "23" smd rect
@@
             (size 1.5 0.9)
             (layers "F.Cu" "F.Mask" "F.Paste")
-            (net 21 "line-25")
+            (net 21 "line-14")
         )
         (pad "24" smd rect
@@
             (size 1.5 0.9)
             (layers "F.Cu" "F.Mask" "F.Paste")
-            (net 28 "line-32")
+            (net 28 "line-12")
         )
         (pad "25" smd rect
@@
             (size 1.5 0.9)
             (layers "F.Cu" "F.Mask" "F.Paste")
-            (net 26 "line-11")
+            (net 26 "line-30")
         )
         (pad "26" smd rect
@@
             (size 1.5 0.9)
             (layers "F.Cu" "F.Mask" "F.Paste")
-            (net 19 "line-3")
+            (net 19 "line-9")
         )
         (pad "27" smd rect
@@
             (size 1.5 0.9)
             (layers "F.Cu" "F.Mask" "F.Paste")
-            (net 11 "line-2")
+            (net 11 "line-22")
         )
         (pad "29" smd rect
@@
             (size 1.5 0.9)
             (layers "F.Cu" "F.Mask" "F.Paste")
-            (net 18 "line-34")
+            (net 18 "line-26")
         )
         (pad "30" smd rect
@@
             (size 1.5 0.9)
             (layers "F.Cu" "F.Mask" "F.Paste")
-            (net 22 "line-10")
+            (net 22 "line-28")
         )
         (pad "31" smd rect
@@
             (size 1.5 0.9)
             (layers "F.Cu" "F.Mask" "F.Paste")
-            (net 9 "line-22")
+            (net 9 "line-34")
         )
         (pad "32" smd rect
@@
             (size 1.5 0.9)
             (layers "F.Cu" "F.Mask" "F.Paste")
-            (net 7 "line-7")
+            (net 7 "line-4")
         )
         (pad "33" smd rect
@@
             (size 1.5 0.9)
             (layers "F.Cu" "F.Mask" "F.Paste")
-            (net 13 "line-14")
+            (net 13 "line-5")
         )
         (pad "34" smd rect
@@
             (size 1.5 0.9)
             (layers "F.Cu" "F.Mask" "F.Paste")
-            (net 10 "line-8")
+            (net 10 "line-10")
         )
         (pad "35" smd rect
@@
             (size 1.5 0.9)
             (layers "F.Cu" "F.Mask" "F.Paste")
-            (net 25 "line-27")
+            (net 25 "line-32")
         )
         (pad "36" smd rect
@@
             (size 1.5 0.9)
             (layers "F.Cu" "F.Mask" "F.Paste")
-            (net 24 "line-17")
+            (net 24 "line-21")
         )
         (pad "37" smd rect
@@
             (size 1.5 0.9)
             (layers "F.Cu" "F.Mask" "F.Paste")
-            (net 16 "line-16")
+            (net 16 "line-8")
         )
         (pad "38" smd rect
@@
             (size 1.5 0.9)
             (layers "F.Cu" "F.Mask" "F.Paste")
-            (net 32 "line-5")
+            (net 32 "line-3")
         )
         (pad "39" smd rect
@@
             (size 1.5 0.9)
             (layers "F.Cu" "F.Mask" "F.Paste")
-            (net 15 "line-30")
+            (net 15 "line-23")
         )
         (pad "40" smd rect
@@
             (size 0.79 0.54)
             (layers "F.Cu" "F.Mask" "F.Paste")
-            (net 41 "in")
+            (net 39 "in")
         )
         (pad "2" smd rect
@@
             (size 1.05 0.7)
             (layers "F.Cu" "F.Mask" "F.Paste")
-            (net 41 "in")
+            (net 39 "in")
         )
         (pad "2" smd rect
@@
             (size 1.05 0.7)
             (layers "F.Cu" "F.Mask" "F.Paste")
-            (net 41 "in")
+            (net 39 "in")
         )
         (pad "3" smd rect

Commit message: try with keep netnames enabled
Connections:
- U2 pad 10: line-2 -> line-18
- U2 pad 11: line-20 -> line
- U2 pad 12: line-18 -> line-3
- U2 pad 13: line-15 -> line-20
- U2 pad 14: line-27 -> line-25
- U2 pad 15: line-7 -> line-32
- U2 pad 16: line-24 -> line-4
- U2 pad 17: line-19 -> line-12
- U2 pad 18: line-1 -> line-27
- U2 pad 19: line -> line-10
- U2 pad 20: line-11 -> line-5
- U2 pad 21: line-16 -> line-13
- U2 pad 22: line-17 -> line-24
- U2 pad 23: line-14 -> line-1
- U2 pad 24: line-12 -> line-17
- U2 pad 25: line-30 -> line-9
- U2 pad 26: line-9 -> line-14
- U2 pad 28: line-22 -> line-23
- U2 pad 29: line-26 -> line-31
- U2 pad 30: line-28 -> line-11
- U2 pad 31: line-34 -> line-28
- U2 pad 32: line-4 -> line-7
- U2 pad 33: line-5 -> line-21
- U2 pad 34: line-10 -> line-15
- U2 pad 35: line-32 -> line-33
- U2 pad 36: line-21 -> line-19
- U2 pad 37: line-8 -> line-16
- U2 pad 38: line-3 -> line-30
- U2 pad 39: line-23 -> line-6
- U2 pad 4: line-13 -> line-29
- U2 pad 5: line-31 -> line-26
- U2 pad 6: line-25 -> line-22
- U2 pad 7: line-6 -> line-8
- U2 pad 8: line-29 -> line-2
- U2 pad 9: line-33 -> line-34
Changed lines of the file:
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@@
     )
     (net 0 "")
-    (net 1 "line-15")
-    (net 2 "line-33")
-    (net 3 "line-16")
-    (net 4 "line-11")
-    (net 5 "line-18")
-    (net 6 "line-6")
-    (net 7 "line-4")
-    (net 8 "line-20")
-    (net 9 "line-34")
-    (net 10 "line-10")
-    (net 11 "line-22")
-    (net 12 "line-2")
-    (net 13 "line-5")
+    (net 1 "line-20")
+    (net 2 "line-34")
+    (net 3 "line-13")
+    (net 4 "line-5")
+    (net 5 "line-3")
+    (net 6 "line-8")
+    (net 7 "line-7")
+    (net 8 "line")
+    (net 9 "line-28")
+    (net 10 "line-15")
+    (net 11 "line-23")
+    (net 12 "line-18")
+    (net 13 "line-21")
     (net 14 "out")
-    (net 15 "line-23")
-    (net 16 "line-8")
-    (net 17 "line-13")
-    (net 18 "line-26")
-    (net 19 "line-9")
-    (net 20 "line-27")
-    (net 21 "line-14")
-    (net 22 "line-28")
-    (net 23 "line")
-    (net 24 "line-21")
-    (net 25 "line-32")
-    (net 26 "line-30")
+    (net 15 "line-6")
+    (net 16 "line-16")
+    (net 17 "line-29")
+    (net 18 "line-31")
+    (net 19 "line-14")
+    (net 20 "line-25")
+    (net 21 "line-1")
+    (net 22 "line-11")
+    (net 23 "line-10")
+    (net 24 "line-19")
+    (net 25 "line-33")
+    (net 26 "line-9")
     (net 27 "hv")
-    (net 28 "line-12")
-    (net 29 "line-1")
-    (net 30 "line-29")
-    (net 31 "line-7")
-    (net 32 "line-3")
-    (net 33 "line-19")
-    (net 34 "line-24")
-    (net 35 "line-31")
-    (net 36 "line-25")
-    (net 37 "line-17")
+    (net 28 "line-17")
+    (net 29 "line-27")
+    (net 30 "line-2")
+    (net 31 "line-32")
+    (net 32 "line-30")
+    (net 33 "line-12")
+    (net 34 "line-4")
+    (net 35 "line-26")
+    (net 36 "line-22")
+    (net 37 "line-24")
     (net 38 "gnd")
     (net 39 "in")
@@
             (size 1.5 0.9)
             (layers "F.Cu" "F.Mask" "F.Paste")
-            (net 17 "line-13")
+            (net 17 "line-29")
         )
         (pad "5" smd rect
@@
             (size 1.5 0.9)
             (layers "F.Cu" "F.Mask" "F.Paste")
-            (net 35 "line-31")
+            (net 35 "line-26")
         )
         (pad "6" smd rect
@@
             (size 1.5 0.9)
             (layers "F.Cu" "F.Mask" "F.Paste")
-            (net 36 "line-25")
+            (net 36 "line-22")
         )
         (pad "7" smd rect
@@
             (size 1.5 0.9)
             (layers "F.Cu" "F.Mask" "F.Paste")
-            (net 6 "line-6")
+            (net 6 "line-8")
         )
         (pad "8" smd rect
@@
             (size 1.5 0.9)
             (layers "F.Cu" "F.Mask" "F.Paste")
-            (net 30 "line-29")
+            (net 30 "line-2")
         )
         (pad "9" smd rect
@@
             (size 1.5 0.9)
             (layers "F.Cu" "F.Mask" "F.Paste")
-            (net 2 "line-33")
+            (net 2 "line-34")
         )
         (pad "10" smd rect
@@
             (size 1.5 0.9)
             (layers "F.Cu" "F.Mask" "F.Paste")
-            (net 12 "line-2")
+            (net 12 "line-18")
         )
         (pad "11" smd rect
@@
             (size 1.5 0.9)
             (layers "F.Cu" "F.Mask" "F.Paste")
-            (net 8 "line-20")
+            (net 8 "line")
         )
         (pad "12" smd rect
@@
             (size 1.5 0.9)
             (layers "F.Cu" "F.Mask" "F.Paste")
-            (net 5 "line-18")
+            (net 5 "line-3")
         )
         (pad "13" smd rect
@@
             (size 1.5 0.9)
             (layers "F.Cu" "F.Mask" "F.Paste")
-            (net 1 "line-15")
+            (net 1 "line-20")
         )
         (pad "14" smd rect
@@
             (size 1.5 0.9)
             (layers "F.Cu" "F.Mask" "F.Paste")
-            (net 20 "line-27")
+            (net 20 "line-25")
         )
         (pad "15" smd rect
@@
             (size 1.5 0.9)
             (layers "F.Cu" "F.Mask" "F.Paste")
-            (net 31 "line-7")
+            (net 31 "line-32")
         )
         (pad "16" smd rect
@@
             (size 1.5 0.9)
             (layers "F.Cu" "F.Mask" "F.Paste")
-            (net 34 "line-24")
+            (net 34 "line-4")
         )
         (pad "17" smd rect
@@
             (size 1.5 0.9)
             (layers "F.Cu" "F.Mask" "F.Paste")
-            (net 33 "line-19")
+            (net 33 "line-12")
         )
         (pad "18" smd rect
@@
             (size 1.5 0.9)
             (layers "F.Cu" "F.Mask" "F.Paste")
-            (net 29 "line-1")
+            (net 29 "line-27")
         )
         (pad "19" smd rect
@@
             (size 1.5 0.9)
             (layers "F.Cu" "F.Mask" "F.Paste")
-            (net 23 "line")
+            (net 23 "line-10")
         )
         (pad "20" smd rect
@@
             (size 1.5 0.9)
             (layers "F.Cu" "F.Mask" "F.Paste")
-            (net 4 "line-11")
+            (net 4 "line-5")
         )
         (pad "21" smd rect
@@
             (size 1.5 0.9)
             (layers "F.Cu" "F.Mask" "F.Paste")
-            (net 3 "line-16")
+            (net 3 "line-13")
         )
         (pad "22" smd rect
@@
             (size 1.5 0.9)
             (layers "F.Cu" "F.Mask" "F.Paste")
-            (net 37 "line-17")
+            (net 37 "line-24")
         )
         (pad "23" smd rect
@@
             (size 1.5 0.9)
             (layers "F.Cu" "F.Mask" "F.Paste")
-            (net 21 "line-14")
+            (net 21 "line-1")
         )
         (pad "24" smd rect
@@
             (size 1.5 0.9)
             (layers "F.Cu" "F.Mask" "F.Paste")
-            (net 28 "line-12")
+            (net 28 "line-17")
         )
         (pad "25" smd rect
@@
             (size 1.5 0.9)
             (layers "F.Cu" "F.Mask" "F.Paste")
-            (net 26 "line-30")
+            (net 26 "line-9")
         )
         (pad "26" smd rect
@@
             (size 1.5 0.9)
             (layers "F.Cu" "F.Mask" "F.Paste")
-            (net 19 "line-9")
+            (net 19 "line-14")
         )
         (pad "27" smd rect
@@
             (size 1.5 0.9)
             (layers "F.Cu" "F.Mask" "F.Paste")
-            (net 11 "line-22")
+            (net 11 "line-23")
         )
         (pad "29" smd rect
@@
             (size 1.5 0.9)
             (layers "F.Cu" "F.Mask" "F.Paste")
-            (net 18 "line-26")
+            (net 18 "line-31")
         )
         (pad "30" smd rect
@@
             (size 1.5 0.9)
             (layers "F.Cu" "F.Mask" "F.Paste")
-            (net 22 "line-28")
+            (net 22 "line-11")
         )
         (pad "31" smd rect
@@
             (size 1.5 0.9)
             (layers "F.Cu" "F.Mask" "F.Paste")
-            (net 9 "line-34")
+            (net 9 "line-28")
         )
         (pad "32" smd rect
@@
             (size 1.5 0.9)
             (layers "F.Cu" "F.Mask" "F.Paste")
-            (net 7 "line-4")
+            (net 7 "line-7")
         )
         (pad "33" smd rect
@@
             (size 1.5 0.9)
             (layers "F.Cu" "F.Mask" "F.Paste")
-            (net 13 "line-5")
+            (net 13 "line-21")
         )
         (pad "34" smd rect
@@
             (size 1.5 0.9)
             (layers "F.Cu" "F.Mask" "F.Paste")
-            (net 10 "line-10")
+            (net 10 "line-15")
         )
         (pad "35" smd rect
@@
             (size 1.5 0.9)
             (layers "F.Cu" "F.Mask" "F.Paste")
-            (net 25 "line-32")
+            (net 25 "line-33")
         )
         (pad "36" smd rect
@@
             (size 1.5 0.9)
             (layers "F.Cu" "F.Mask" "F.Paste")
-            (net 24 "line-21")
+            (net 24 "line-19")
         )
         (pad "37" smd rect
@@
             (size 1.5 0.9)
             (layers "F.Cu" "F.Mask" "F.Paste")
-            (net 16 "line-8")
+            (net 16 "line-16")
         )
         (pad "38" smd rect
@@
             (size 1.5 0.9)
             (layers "F.Cu" "F.Mask" "F.Paste")
-            (net 32 "line-3")
+            (net 32 "line-30")
         )
         (pad "39" smd rect
@@
             (size 1.5 0.9)
             (layers "F.Cu" "F.Mask" "F.Paste")
-            (net 15 "line-23")
+            (net 15 "line-6")
         )
         (pad "40" smd rect
