File: packages/esp32s3/layouts/esp32_s3_wroom_reference_design/esp32_s3_wroom_reference_design.kicad_pcb (KiCad board)
At the start: 2 copper layers, 7 parts

Commit message: Update with new ato 0.7.x features
Connections:
- net in renamed input
- net out renamed output
- U2 pad 10: line-18 -> line-29
- U2 pad 11: line -> line-22
- U2 pad 12: line-3 -> line-16
- U2 pad 13: line-20 -> line
- U2 pad 14: line-25 -> line-18
- U2 pad 15: line-32 -> line-7
- U2 pad 16: line-4 -> line-17
- U2 pad 17: line-12 -> line-14
- U2 pad 18: line-27 -> line-4
- U2 pad 19: line-10 -> line-34
- U2 pad 20: line-5 -> line-23
- U2 pad 21: line-13 -> line-6
- U2 pad 22: line-24 -> line-33
- U2 pad 23: line-1 -> line-2
- U2 pad 24: line-17 -> line-30
- U2 pad 25: line-9 -> line-19
- U2 pad 26: line-14 -> line-10
- U2 pad 28: line-23 -> line-15
- U2 pad 29: line-31 -> line-25
- U2 pad 30: line-11 -> line-13
- U2 pad 31: line-28 -> line-20
- U2 pad 32: line-7 -> line-1
- U2 pad 33: line-21 -> line-28
- U2 pad 34: line-15 -> line-27
- U2 pad 35: line-33 -> line-31
- U2 pad 36: line-19 -> line-8
- U2 pad 37: line-16 -> line-3
- U2 pad 38: line-30 -> line-21
- U2 pad 39: line-6 -> line-11
- U2 pad 4: line-29 -> line-12
- U2 pad 6: line-22 -> line-5
- U2 pad 7: line-8 -> line-24
- U2 pad 8: line-2 -> line-32
- U2 pad 9: line-34 -> line-9
Changed lines of the file:
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@@
     )
     (net 0 "")
-    (net 1 "line-20")
-    (net 2 "line-34")
-    (net 3 "line-13")
-    (net 4 "line-5")
-    (net 5 "line-3")
-    (net 6 "line-8")
-    (net 7 "line-7")
-    (net 8 "line")
-    (net 9 "line-28")
-    (net 10 "line-15")
-    (net 11 "line-23")
-    (net 12 "line-18")
-    (net 13 "line-21")
-    (net 14 "out")
-    (net 15 "line-6")
-    (net 16 "line-16")
-    (net 17 "line-29")
-    (net 18 "line-31")
-    (net 19 "line-14")
-    (net 20 "line-25")
-    (net 21 "line-1")
-    (net 22 "line-11")
-    (net 23 "line-10")
-    (net 24 "line-19")
-    (net 25 "line-33")
-    (net 26 "line-9")
+    (net 1 "line")
+    (net 2 "line-9")
+    (net 3 "line-6")
+    (net 4 "line-23")
+    (net 5 "line-16")
+    (net 6 "line-24")
+    (net 7 "line-1")
+    (net 8 "line-22")
+    (net 9 "line-20")
+    (net 10 "line-27")
+    (net 11 "line-15")
+    (net 12 "line-29")
+    (net 13 "line-28")
+    (net 14 "output")
+    (net 15 "line-11")
+    (net 16 "line-3")
+    (net 17 "line-12")
+    (net 18 "line-25")
+    (net 19 "line-10")
+    (net 20 "line-18")
+    (net 21 "line-2")
+    (net 22 "line-13")
+    (net 23 "line-34")
+    (net 24 "line-8")
+    (net 25 "line-31")
+    (net 26 "line-19")
     (net 27 "hv")
-    (net 28 "line-17")
-    (net 29 "line-27")
-    (net 30 "line-2")
-    (net 31 "line-32")
-    (net 32 "line-30")
-    (net 33 "line-12")
-    (net 34 "line-4")
+    (net 28 "line-30")
+    (net 29 "line-4")
+    (net 30 "line-32")
+    (net 31 "line-7")
+    (net 32 "line-21")
+    (net 33 "line-14")
+    (net 34 "line-17")
     (net 35 "line-26")
-    (net 36 "line-22")
-    (net 37 "line-24")
+    (net 36 "line-5")
+    (net 37 "line-33")
     (net 38 "gnd")
-    (net 39 "in")
+    (net 39 "input")
     (footprint "atopile:R0402-56259e"
         (layer "F.Cu")
@@
             (size 0.57 0.54)
             (layers "F.Cu" "F.Mask" "F.Paste")
-            (net 39 "in")
+            (net 39 "input")
         )
         (embedded_fonts no)
@@
             (size 1.5 0.9)
             (layers "F.Cu" "F.Mask" "F.Paste")
-            (net 39 "in")
+            (net 39 "input")
         )
         (pad "4" smd rect
@@
             (size 1.5 0.9)
             (layers "F.Cu" "F.Mask" "F.Paste")
-            (net 17 "line-29")
+            (net 17 "line-12")
         )
         (pad "5" smd rect
@@
             (size 1.5 0.9)
             (layers "F.Cu" "F.Mask" "F.Paste")
-            (net 36 "line-22")
+            (net 36 "line-5")
         )
         (pad "7" smd rect
@@
             (size 1.5 0.9)
             (layers "F.Cu" "F.Mask" "F.Paste")
-            (net 6 "line-8")
+            (net 6 "line-24")
         )
         (pad "8" smd rect
@@
             (size 1.5 0.9)
             (layers "F.Cu" "F.Mask" "F.Paste")
-            (net 30 "line-2")
+            (net 30 "line-32")
         )
         (pad "9" smd rect
@@
             (size 1.5 0.9)
             (layers "F.Cu" "F.Mask" "F.Paste")
-            (net 2 "line-34")
+            (net 2 "line-9")
         )
         (pad "10" smd rect
@@
             (size 1.5 0.9)
             (layers "F.Cu" "F.Mask" "F.Paste")
-            (net 12 "line-18")
+            (net 12 "line-29")
         )
         (pad "11" smd rect
@@
             (size 1.5 0.9)
             (layers "F.Cu" "F.Mask" "F.Paste")
-            (net 8 "line")
+            (net 8 "line-22")
         )
         (pad "12" smd rect
@@
             (size 1.5 0.9)
             (layers "F.Cu" "F.Mask" "F.Paste")
-            (net 5 "line-3")
+            (net 5 "line-16")
         )
         (pad "13" smd rect
@@
             (size 1.5 0.9)
             (layers "F.Cu" "F.Mask" "F.Paste")
-            (net 1 "line-20")
+            (net 1 "line")
         )
         (pad "14" smd rect
@@
             (size 1.5 0.9)
             (layers "F.Cu" "F.Mask" "F.Paste")
-            (net 20 "line-25")
+            (net 20 "line-18")
         )
         (pad "15" smd rect
@@
             (size 1.5 0.9)
             (layers "F.Cu" "F.Mask" "F.Paste")
-            (net 31 "line-32")
+            (net 31 "line-7")
         )
         (pad "16" smd rect
@@
             (size 1.5 0.9)
             (layers "F.Cu" "F.Mask" "F.Paste")
-            (net 34 "line-4")
+            (net 34 "line-17")
         )
         (pad "17" smd rect
@@
             (size 1.5 0.9)
             (layers "F.Cu" "F.Mask" "F.Paste")
-            (net 33 "line-12")
+            (net 33 "line-14")
         )
         (pad "18" smd rect
@@
             (size 1.5 0.9)
             (layers "F.Cu" "F.Mask" "F.Paste")
-            (net 29 "line-27")
+            (net 29 "line-4")
         )
         (pad "19" smd rect
@@
             (size 1.5 0.9)
             (layers "F.Cu" "F.Mask" "F.Paste")
-            (net 23 "line-10")
+            (net 23 "line-34")
         )
         (pad "20" smd rect
@@
             (size 1.5 0.9)
             (layers "F.Cu" "F.Mask" "F.Paste")
-            (net 4 "line-5")
+            (net 4 "line-23")
         )
         (pad "21" smd rect
@@
             (size 1.5 0.9)
             (layers "F.Cu" "F.Mask" "F.Paste")
-            (net 3 "line-13")
+            (net 3 "line-6")
         )
         (pad "22" smd rect
@@
             (size 1.5 0.9)
             (layers "F.Cu" "F.Mask" "F.Paste")
-            (net 37 "line-24")
+            (net 37 "line-33")
         )
         (pad "23" smd rect
@@
             (size 1.5 0.9)
             (layers "F.Cu" "F.Mask" "F.Paste")
-            (net 21 "line-1")
+            (net 21 "line-2")
         )
         (pad "24" smd rect
@@
             (size 1.5 0.9)
             (layers "F.Cu" "F.Mask" "F.Paste")
-            (net 28 "line-17")
+            (net 28 "line-30")
         )
         (pad "25" smd rect
@@
             (size 1.5 0.9)
             (layers "F.Cu" "F.Mask" "F.Paste")
-            (net 26 "line-9")
+            (net 26 "line-19")
         )
         (pad "26" smd rect
@@
             (size 1.5 0.9)
             (layers "F.Cu" "F.Mask" "F.Paste")
-            (net 19 "line-14")
+            (net 19 "line-10")
         )
         (pad "27" smd rect
@@
             (size 1.5 0.9)
             (layers "F.Cu" "F.Mask" "F.Paste")
-            (net 14 "out")
+            (net 14 "output")
         )
         (pad "28" smd rect
@@
             (size 1.5 0.9)
             (layers "F.Cu" "F.Mask" "F.Paste")
-            (net 11 "line-23")
+            (net 11 "line-15")
         )
         (pad "29" smd rect
@@
             (size 1.5 0.9)
             (layers "F.Cu" "F.Mask" "F.Paste")
-            (net 18 "line-31")
+            (net 18 "line-25")
         )
         (pad "30" smd rect
@@
             (size 1.5 0.9)
             (layers "F.Cu" "F.Mask" "F.Paste")
-            (net 22 "line-11")
+            (net 22 "line-13")
         )
         (pad "31" smd rect
@@
             (size 1.5 0.9)
             (layers "F.Cu" "F.Mask" "F.Paste")
-            (net 9 "line-28")
+            (net 9 "line-20")
         )
         (pad "32" smd rect
@@
             (size 1.5 0.9)
             (layers "F.Cu" "F.Mask" "F.Paste")
-            (net 7 "line-7")
+            (net 7 "line-1")
         )
         (pad "33" smd rect
@@
             (size 1.5 0.9)
             (layers "F.Cu" "F.Mask" "F.Paste")
-            (net 13 "line-21")
+            (net 13 "line-28")
         )
         (pad "34" smd rect
@@
             (size 1.5 0.9)
             (layers "F.Cu" "F.Mask" "F.Paste")
-            (net 10 "line-15")
+            (net 10 "line-27")
         )
         (pad "35" smd rect
@@
             (size 1.5 0.9)
             (layers "F.Cu" "F.Mask" "F.Paste")
-            (net 25 "line-33")
+            (net 25 "line-31")
         )
         (pad "36" smd rect
@@
             (size 1.5 0.9)
             (layers "F.Cu" "F.Mask" "F.Paste")
-            (net 24 "line-19")
+            (net 24 "line-8")
         )
         (pad "37" smd rect
@@
             (size 1.5 0.9)
             (layers "F.Cu" "F.Mask" "F.Paste")
-            (net 16 "line-16")
+            (net 16 "line-3")
         )
         (pad "38" smd rect
@@
             (size 1.5 0.9)
             (layers "F.Cu" "F.Mask" "F.Paste")
-            (net 32 "line-30")
+            (net 32 "line-21")
         )
         (pad "39" smd rect
@@
             (size 1.5 0.9)
             (layers "F.Cu" "F.Mask" "F.Paste")
-            (net 15 "line-6")
+            (net 15 "line-11")
         )
         (pad "40" smd rect
@@
             (size 1.05 0.7)
             (layers "F.Cu" "F.Mask" "F.Paste")
-            (net 14 "out")
+            (net 14 "output")
         )
         (pad "4" smd rect
@@
             (size 1.05 0.7)
             (layers "F.Cu" "F.Mask" "F.Paste")
-            (net 14 "out")
+            (net 14 "output")
         )
         (embedded_fonts no)
@@
             (size 0.79 0.54)
             (layers "F.Cu" "F.Mask" "F.Paste")
-            (net 39 "in")
+            (net 39 "input")
         )
         (pad "2" smd rect
@@
             (size 1.05 0.7)
             (layers "F.Cu" "F.Mask" "F.Paste")
-            (net 39 "in")
+            (net 39 "input")
         )
         (pad "2" smd rect
@@
             (size 1.05 0.7)
             (layers "F.Cu" "F.Mask" "F.Paste")
-            (net 39 "in")
+            (net 39 "input")
         )
         (pad "3" smd rect

Commit message: Fix missing connection between JTAG and reset (enable)
Connections:
- U2 pad 10: line-29 -> line-25
- U2 pad 11: line-22 -> line-18
- U2 pad 12: line-16 -> line-26
- U2 pad 14: line-18 -> line-29
- U2 pad 15: line-7 -> line-31
- U2 pad 16: line-17 -> line-5
- U2 pad 17: line-14 -> line-12
- U2 pad 18: line-4 -> line-34
- U2 pad 19: line-34 -> line-3
- U2 pad 20: line-23 -> line-9
- U2 pad 21: line-6 -> line-7
- U2 pad 22: line-33 -> line-16
- U2 pad 23: line-2 -> line-32
- U2 pad 24: line-30 -> line-2
- U2 pad 25: line-19 -> line-20
- U2 pad 26: line-10 -> line-4
- U2 pad 28: line-15 -> line-6
- U2 pad 29: line-25 -> line-22
- U2 pad 30: line-13 -> line-1
- U2 pad 31: line-20 -> line-15
- U2 pad 32: line-1 -> line-11
- U2 pad 33: line-28 -> line-14
- U2 pad 34: line-27 -> line-19
- U2 pad 35: line-31 -> line-30
- U2 pad 37: line-3 -> line-17
- U2 pad 38: line-21 -> line-10
- U2 pad 39: line-11 -> line-23
- U2 pad 4: line-12 -> line-21
- U2 pad 5: line-26 -> line-13
- U2 pad 6: line-5 -> line-24
- U2 pad 7: line-24 -> line-33
- U2 pad 8: line-32 -> line-28
- U2 pad 9: line-9 -> line-27
Routing:
- net input: track 0.00 -> 10.2 mm
- net (no net): track 10.2 -> 0.00 mm
