File: packages/esp32c3/layouts/esp32_c3_mini_ufl_reference_design/esp32_c3_mini_ufl_reference_design.kicad_pcb (KiCad board)
At the start: 2 copper layers, 9 parts

Commit message: Connect extra gnd pins
Connections:
- C3 pad 1: output-1 -> output
- R1 pad 1: line -> line-3
- R2 pad 1: line-1 -> line-11
- R3 pad 2: output-1 -> output
- U1 pad 3: output -> output-1
- U1 pad 4: output -> output-1
- U2 pad 13: line-7 -> line
- U2 pad 16: line-4 -> line-12
- U2 pad 18: line-2 -> line-7
- U2 pad 19: line-3 -> line-8
- U2 pad 20: line-5 -> line-2
- U2 pad 21: line-6 -> line-9
- U2 pad 22: line-1 -> line-11
- U2 pad 23: output -> output-1
- U2 pad 26: line-9 -> line-10
- U2 pad 27: line-10 -> line-1
- U2 pad 30: line-8 -> line-4
- U2 pad 31: line-12 -> line-5
- U2 pad 5: line -> line-3
- U2 pad 6: line-11 -> line-6
- U2 pad 8: output-1 -> output
- U3 pad 3: output-1 -> output
- U3 pad 4: output-1 -> output
Routing:
- net output-1: track 10.1 -> 1.63 mm
- net output: track 1.63 -> 10.1 mm
- net line-11: track 0.00 -> 5.04 mm
- net line-1: track 5.04 -> 0.00 mm
- net line-3: track 0.00 -> 2.67 mm
- net line: track 2.67 -> 0.00 mm

Commit message: Update packages:
- requited
- package > driver method
- cleaning up
- aligning packages
Parts:
- removed C1: 22µF ±20% 6.3V X5R, atopile:C0603-bd72f6
- removed C2: 100nF ±10% 16V X7R, atopile:C0402-b3ef17
- removed C3: 1µF ±10% 25V X5R, atopile:C0402-b3ef17
- removed R1, R2, R3: 10kΩ ±1% 62.5mW, atopile:R0402-56259e
- removed U1, U3: , lib:KEY-SMD_4P-L4.2-W3.2-P2.20-LS4.6
- removed U2: , atopile:WIFIM-SMD_ESP32-C3-MINI-MINI-1U-1cb675
Routing:
- net output: track 10.1 -> 0.00 mm
- net hv: track 6.55 -> 0.00 mm
- net gnd: track 5.11 -> 0.00 mm
- net line-11: track 5.04 -> 0.00 mm
- net line-3: track 2.67 -> 0.00 mm
- net output-1: track 1.63 -> 0.00 mm
- removed copper zone on B.Cu, net gnd
- removed copper zone on F.Cu, net gnd
