File: packages/usb/layouts/usb_pd_power_sink/usb_pd_power_sink.kicad_pcb (KiCad board)
At the start: 2 copper layers, 8 parts

Commit message: Rebuild usb package
Connections:
- net DP1 renamed DP2
- R2 pad 2: pd_trigger-line-1 -> pd_trigger-line
- R4 pad 1: pd_trigger-line -> pd_trigger-line-1
- U1 pad 2: pd_trigger.controller-line -> pd_trigger.controller-line-1
- U1 pad 3: pd_trigger.controller-line-1 -> pd_trigger.controller-line
- U1 pad 8: pd_trigger-line-1 -> pd_trigger-line
- U1 pad 9: pd_trigger-line -> pd_trigger-line-1

Commit message: Rebuild all
Connections:
- R2 pad 2: pd_trigger-line -> pd_trigger-line-1
- R4 pad 1: pd_trigger-line-1 -> pd_trigger-line
- U1 pad 8: pd_trigger-line -> pd_trigger-line-1
- U1 pad 9: pd_trigger-line-1 -> pd_trigger-line
Changed lines of the file:
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@@
     (net 7 "line-1")
     (net 8 "line")
-    (net 9 "pd_trigger-line")
+    (net 9 "pd_trigger-line-1")
     (net 10 "hv")
-    (net 11 "pd_trigger-line-1")
+    (net 11 "pd_trigger-line")
     (net 12 "anode")
     (net 13 "pd_trigger-gnd")
@@
             (size 0.57 0.54)
             (layers "F.Cu" "F.Mask" "F.Paste")
-            (net 11 "pd_trigger-line-1")
+            (net 11 "pd_trigger-line")
         )
         (pad "2" smd rect
@@
             (size 1.5 0.6)
             (layers "F.Cu" "F.Mask" "F.Paste")
-            (net 9 "pd_trigger-line")
+            (net 9 "pd_trigger-line-1")
         )
         (pad "9" smd rect
@@
             (size 1.5 0.6)
             (layers "F.Cu" "F.Mask" "F.Paste")
-            (net 11 "pd_trigger-line-1")
+            (net 11 "pd_trigger-line")
         )
         (pad "10" smd rect
@@
             (size 0.57 0.54)
             (layers "F.Cu" "F.Mask" "F.Paste")
-            (net 9 "pd_trigger-line")
+            (net 9 "pd_trigger-line-1")
         )
         (embedded_fonts no)
