File: packages/logos/layouts/test/test.kicad_pcb (KiCad board)
At the start: 2 copper layers, 1 part

Commit message: WIP update packages till ESPs
Parts:
- LOGO1: footprint lib:faebrykLogo_8x9mm -> faebryk_Logo_8x9mm:faebryk_Logo_8x9mm
Changed lines of the file:
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@@
     (version 20241229)
     (generator "atopile")
-    (generator_version "0.5.0")
+    (generator_version "0.9.0")
     (general
         (thickness 1.6)
@@
     )
     (net 0 "")
-    (footprint "lib:faebrykLogo_8x9mm"
+    (footprint "faebryk_Logo_8x9mm:faebryk_Logo_8x9mm"
         (layer "F.Cu")
         (at 0 0 0)
@@
             )
         )
-        (property "__atopile_lib_fp_hash__" "f2bdc385-8507-a988-77cc-0c8e09ebc3de"
+        (property "__atopile_lib_fp_hash__" "22d7f1ae-c8f4-5b6d-718f-fa8e9b31326c"
             (at 0 0 0)
             (layer "User.9")
@@
             )
         )
-        (property "atopile_address" ""
+        (property "atopile_address" "logo"
             (at 0 0 0)
             (layer "User.9")
@@
         )
         (attr board_only exclude_from_pos_files exclude_from_bom)
-        (fp_text user "FBRK:autoplaced"
-            (at 0 0 0)
-            (layer "User.5")
-            (effects
-                (font
-                    (size 0.125 0.125)
-                    (thickness 0.01875)
-                )
-                (hide no)
-            )
-            (unlocked no)
-        )
         (fp_poly
             (pts
