File: packages/connectors/layouts/qwiic_horizontal/qwiic_horizontal.kicad_pcb (KiCad board)
At the start: 2 copper layers, 2 parts

Commit message: Rebuild all
Connections:
- CN1 pad 3: line -> line-1
- CN1 pad 4: line-1 -> line
Changed lines of the file:
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@@
     (net 0 "")
     (net 2 "hv")
-    (net 4 "line-1")
-    (net 6 "line")
+    (net 4 "line")
+    (net 6 "line-1")
     (net 7 "gnd")
     (footprint "atopile:CONN-SMD_4P-P1.00_SM04B-SRSS-TB-LF-SN-d36980"
@@
             (size 0.6 1.55)
             (layers "F.Cu" "F.Mask" "F.Paste")
-            (net 6 "line")
+            (net 6 "line-1")
         )
         (pad "4" smd rect
@@
             (size 0.6 1.55)
             (layers "F.Cu" "F.Mask" "F.Paste")
-            (net 4 "line-1")
+            (net 4 "line")
         )
         (pad "5" smd rect

Commit message: WIP update connectors
Parts:
- U1: footprint lib:qwiic_6mm -> atopile:qwiic_6mm
Changed lines of the file:
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@@
         (embedded_fonts no)
     )
-    (footprint "lib:qwiic_6mm"
+    (footprint "atopile:qwiic_6mm"
         (layer "F.Cu")
         (at 0 -4.25 0)

Commit message: WIP update packages till ESPs
Parts:
- CN1: footprint atopile:CONN-SMD_4P-P1.00_SM04B-SRSS-TB-LF-SN-d36980 -> JST_Sales_America_SM04B_SRSS_TB_LF__SN:CONN-SMD_4P-P1.00_SM04B-SRSS-TB-LF-SN
- U1: footprint atopile:qwiic_6mm -> Sparkfun_QWIIC_Logo:qwiic_6mm
Connections:
- CN1 pad 3: line-1 -> line
- CN1 pad 4: line -> line-1
Changed lines of the file:
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@@
     )
     (net 0 "")
-    (net 2 "hv")
-    (net 4 "line")
-    (net 6 "line-1")
-    (net 7 "gnd")
-    (footprint "atopile:CONN-SMD_4P-P1.00_SM04B-SRSS-TB-LF-SN-d36980"
+    (net 1 "hv")
+    (net 2 "line-1")
+    (net 3 "line")
+    (net 4 "gnd")
+    (footprint "JST_Sales_America_SM04B_SRSS_TB_LF__SN:CONN-SMD_4P-P1.00_SM04B-SRSS-TB-LF-SN"
         (layer "F.Cu")
         (at 0 0 0)
@@
         (property "Datasheet" "https://www.lcsc.com/datasheet/lcsc_datasheet_2304140030_JST-SM04B-SRSS-TB-LF-SN_C160404.pdf"
             (at 0 0 0)
-            (layer "User.9")
-            (hide yes)
-            (effects
-                (font
-                    (size 0.125 0.125)
-                    (thickness 0.01875)
+            (layer "F.Fab")
+            (hide yes)
+            (effects
+                (font
+                    (size 1.27 1.27)
+                    (thickness 0.15)
                 )
             )
@@
             )
         )
-        (property "__atopile_lib_fp_hash__" "227254e0-5a73-7ef2-aacf-83e6b9bc6961"
+        (property "checksum" "005e6dc3038a599246199d51285475b6bd6f6dbc0b1845e8c7ea0725bfb4faea"
+            (at 0 0 0)
+            (layer "User.9")
+            (hide yes)
+            (effects
+                (font
+                    (size 0.125 0.125)
+                    (thickness 0.01875)
+                )
+            )
+        )
+        (property "__atopile_lib_fp_hash__" "daaac122-8194-c9c6-07d4-e25da2aa4e39"
             (at 0 0 0)
             (layer "User.9")
@@
         )
         (fp_text user "${REFERENCE}"
+            (at 0 -5.94 0)
+            (layer "F.SilkS")
+            (effects
+                (font
+                    (size 1 1)
+                    (thickness 0.15)
+                )
+                (hide yes)
+            )
+            (unlocked no)
+        )
+        (fp_text user "${REFERENCE}"
             (at 0 0 0)
             (layer "F.Fab")
@@
             (size 0.6 1.55)
             (layers "F.Cu" "F.Mask" "F.Paste")
-            (net 7 "gnd")
+            (net 4 "gnd")
         )
         (pad "2" smd rect
@@
             (size 0.6 1.55)
             (layers "F.Cu" "F.Mask" "F.Paste")
-            (net 2 "hv")
+            (net 1 "hv")
         )
         (pad "3" smd rect
@@
             (size 0.6 1.55)
             (layers "F.Cu" "F.Mask" "F.Paste")
-            (net 6 "line-1")
+            (net 3 "line")
         )
         (pad "4" smd rect
@@
             (size 0.6 1.55)
             (layers "F.Cu" "F.Mask" "F.Paste")
-            (net 4 "line")
+            (net 2 "line-1")
         )
         (pad "5" smd rect
@@
             (size 1.2 1.8)
             (layers "F.Cu" "F.Mask" "F.Paste")
-            (net 7 "gnd")
+            (net 4 "gnd")
         )
         (pad "6" smd rect
@@
             (size 1.2 1.8)
             (layers "F.Cu" "F.Mask" "F.Paste")
-            (net 7 "gnd")
+            (net 4 "gnd")
         )
         (embedded_fonts no)
+        (model "${KIPRJMOD}/../../parts/JST_Sales_America_SM04B_SRSS_TB_LF__SN/CONN-SMD_SR1.00-WS-4P.step"
+            (offset
+                (xyz -1.5 -0.5 0)
+            )
+            (scale
+                (xyz 1 1 1)
+            )
+            (rotate
+                (xyz 0 0 0)
+            )
+        )
     )
-    (footprint "atopile:qwiic_6mm"
+    (footprint "Sparkfun_QWIIC_Logo:qwiic_6mm"
         (layer "F.Cu")
         (at 0 -4.25 0)
@@
             )
         )
-        (property "__atopile_lib_fp_hash__" "87d7182d-7b52-4911-551d-73de866a7f5a"
-            (at 0 0 0)
-            (layer "User.9")
+        (property "__atopile_lib_fp_hash__" "d5134a8f-6d12-92b9-05fc-770d84a722a0"
+            (at 0 0 0)
+            (layer "User.9")
