File: packages/connectors/layouts/dual_banana_connectors/dual_banana_connectors.kicad_pcb (KiCad board)
At the start: 2 copper layers, 2 parts

Commit message: Add QWIIC to connector package
Connections:
- J1 pad 1: black_plug-net-3 -> black_plug-net-2
- J1 pad 2: black_plug-net-2 -> black_plug-net-3
- J2 pad 1: red_plug-net -> red_plug-net-3
- J2 pad 2: red_plug-net-1 -> red_plug-net-2
- J2 pad 3: red_plug-net-2 -> red_plug-net-1
- J2 pad 4: red_plug-net-3 -> red_plug-net

Commit message: Rebuild all
Connections:
- J1 pad 2: black_plug-net-3 -> black_plug-net
- J1 pad 3: black_plug-net -> black_plug-net-3
- J2 pad 1: red_plug-net-3 -> red_plug-net-1
- J2 pad 2: red_plug-net-2 -> red_plug-net-3
- J2 pad 3: red_plug-net-1 -> red_plug-net
- J2 pad 4: red_plug-net -> red_plug-net-2
Changed lines of the file:
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@@
     )
     (net 0 "")
-    (net 1 "black_plug-net-3")
-    (net 2 "red_plug-net-1")
-    (net 3 "red_plug-net-3")
+    (net 1 "black_plug-net")
+    (net 2 "red_plug-net")
+    (net 3 "red_plug-net-1")
     (net 4 "black_plug-net-2")
     (net 5 "black_plug-net-1")
-    (net 6 "black_plug-net")
+    (net 6 "black_plug-net-3")
     (net 7 "gnd")
-    (net 8 "red_plug-net-2")
+    (net 8 "red_plug-net-3")
     (net 9 "hv")
-    (net 10 "red_plug-net")
+    (net 10 "red_plug-net-2")
     (footprint "atopile:ANT-TH_L33.0-W12.0_RED-b58375"
         (layer "F.Cu")
@@
             (drill 1.300023)
             (layers "*.Cu" "*.Mask")
-            (net 3 "red_plug-net-3")
+            (net 3 "red_plug-net-1")
             (remove_unused_layers no)
         )
@@
             (drill 1.300023)
             (layers "*.Cu" "*.Mask")
-            (net 8 "red_plug-net-2")
+            (net 8 "red_plug-net-3")
             (remove_unused_layers no)
         )
@@
             (drill 1.300023)
             (layers "*.Cu" "*.Mask")
-            (net 2 "red_plug-net-1")
+            (net 2 "red_plug-net")
             (remove_unused_layers no)
         )
@@
             (drill 1.300023)
             (layers "*.Cu" "*.Mask")
-            (net 10 "red_plug-net")
+            (net 10 "red_plug-net-2")
             (remove_unused_layers no)
         )
@@
             )
         )
-        (property "Datasheet" "https://wmsc.lcsc.com/wmsc/upload/file/pdf/v2/lcsc/2307211803_Changzhou-Amass-Elec-24-245-2_C7437327.pdf"
+        (property "Datasheet" "https://wmsc.lcsc.com/wmsc/upload/file/pdf/v2/lcsc/2307191746_Changzhou-Amass-Elec-24-245-1_C7437326.pdf"
             (at 0 0 90)
             (layer "User.9")
@@
             (drill 1.799996)
             (layers "*.Cu" "*.Mask")
-            (net 1 "black_plug-net-3")
+            (net 1 "black_plug-net")
             (remove_unused_layers no)
         )
@@
             (drill 1.799996)
             (layers "*.Cu" "*.Mask")
-            (net 6 "black_plug-net")
-            (remove_unused_layers no)
-        )
+            (net 6 "black_plug-net-3")
+            (remove_unused_layers no)
+        )

Commit message: WIP update connectors
Parts:
- J1: footprint atopile:ANT-TH_L33.0-W12.0_BLACK-6b51ce -> Changzhou_Amass_Elec_24_245_2:ANT-TH_L33.0-W12.0_BLACK
- J2: footprint atopile:ANT-TH_L33.0-W12.0_RED-b58375 -> Changzhou_Amass_Elec_24_245_1:ANT-TH_L33.0-W12.0_RED
Connections:
- J1 pad 1: black_plug-net-2 -> black_plug-net-1
- J1 pad 4: black_plug-net-1 -> black_plug-net-2
- J2 pad 1: red_plug-net-1 -> red_plug-net-3
- J2 pad 2: red_plug-net-3 -> red_plug-net-2
- J2 pad 3: red_plug-net -> red_plug-net-1
- J2 pad 4: red_plug-net-2 -> red_plug-net

Commit message: WIP update packages till ESPs
Connections:
- J1 pad 1: black_plug-net-1 -> black_plug-net
- J1 pad 2: black_plug-net -> black_plug-net-1
- J1 pad 3: black_plug-net-3 -> black_plug-net-2
- J1 pad 4: black_plug-net-2 -> black_plug-net-3
- J2 pad 2: red_plug-net-2 -> red_plug-net-1
- J2 pad 3: red_plug-net-1 -> red_plug-net
- J2 pad 4: red_plug-net -> red_plug-net-2

Commit message: Manually fix fp lib tables
fix some small bugs
fix package only modules (e.g. logos)
Connections:
- J1 pad 1: black_plug-net -> black_plug-net-1
- J1 pad 2: black_plug-net-1 -> black_plug-net-3
- J1 pad 4: black_plug-net-3 -> black_plug-net
- J2 pad 2: red_plug-net-1 -> red_plug-net-2
- J2 pad 4: red_plug-net-2 -> red_plug-net-1
Changed lines of the file:
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@@
     )
     (net 0 "")
-    (net 1 "black_plug-net-1")
+    (net 1 "black_plug-net-3")
     (net 2 "red_plug-net")
     (net 3 "red_plug-net-3")
-    (net 4 "black_plug-net")
-    (net 5 "black_plug-net-3")
+    (net 4 "black_plug-net-1")
+    (net 5 "black_plug-net")
     (net 6 "black_plug-net-2")
     (net 7 "gnd")
-    (net 8 "red_plug-net-1")
+    (net 8 "red_plug-net-2")
     (net 9 "hv")
-    (net 10 "red_plug-net-2")
+    (net 10 "red_plug-net-1")
     (footprint "Changzhou_Amass_Elec_24_245_1:ANT-TH_L33.0-W12.0_RED"
         (layer "F.Cu")
@@
             (drill 1.300023)
             (layers "*.Cu" "*.Mask")
-            (net 8 "red_plug-net-1")
+            (net 8 "red_plug-net-2")
             (remove_unused_layers no)
         )
@@
             (drill 1.300023)
             (layers "*.Cu" "*.Mask")
-            (net 10 "red_plug-net-2")
+            (net 10 "red_plug-net-1")
             (remove_unused_layers no)
         )
@@
             (drill 1.799996)
             (layers "*.Cu" "*.Mask")
-            (net 4 "black_plug-net")
+            (net 4 "black_plug-net-1")
             (remove_unused_layers no)
         )
@@
             (drill 1.799996)
             (layers "*.Cu" "*.Mask")
-            (net 1 "black_plug-net-1")
+            (net 1 "black_plug-net-3")
             (remove_unused_layers no)
         )
@@
             (drill 1.799996)
             (layers "*.Cu" "*.Mask")
-            (net 5 "black_plug-net-3")
-            (remove_unused_layers no)
-        )
+            (net 5 "black_plug-net")
+            (remove_unused_layers no)
+        )

Commit message: rebuild all packages & regenerate images of changed layouts (silk)
Add new scripts for version bump and build (based on atopile/packages)
Connections:
- net black_plug-net renamed black_plug-_4
- net black_plug-net-1 renamed black_plug-_1
- net black_plug-net-2 renamed black_plug-_3
- net black_plug-net-3 renamed black_plug-_2
- net red_plug-net renamed red_plug-_3
- net red_plug-net-1 renamed red_plug-_4
- net red_plug-net-2 renamed red_plug-_2
- net red_plug-net-3 renamed red_plug-_1
