File: packages/connectors/layouts/qwiic_vertical/qwiic_vertical.kicad_pcb (KiCad board)
At the start: 2 copper layers, 2 parts

Commit message: WIP update packages till ESPs
Parts:
- CN1: footprint atopile:CONN-SMD_BM04B-SRSS-TB-6963ef -> JST_Sales_America_BM04B_SRSS_TB_LF__SN:CONN-SMD_BM04B-SRSS-TB
- U1: footprint lib:qwiic_6mm -> Sparkfun_QWIIC_Logo:qwiic_6mm

Commit message: rebuild all packages & regenerate images of changed layouts (silk)
Add new scripts for version bump and build (based on atopile/packages)
Connections:
- CN1 pad 3: line-1 -> line
- CN1 pad 4: line -> line-1
