File: packages/debug-interfaces/layouts/segger_jlink_compact/segger_jlink_compact.kicad_pcb (KiCad board)
At the start: 2 copper layers, 4 parts

Commit message: WIP update packages till ESPs
Parts:
- H1, H2: footprint atopile:SMD_BD5.6-L5.6-W5.6-D4.1-1d1819 -> Sinhoo_SMTSO2530CTJ:SMD_BD5.6-L5.6-W5.6-D4.1
- J1: footprint atopile:CONN-SMD_20P-P2.54_BH-00019-f2b3b5 -> Liansheng_BH_00019:CONN-SMD_20P-P2.54_BH-00019
- MOD1: footprint lib:segger_jlink_compact -> SEGGER_JLink_Compact:segger_jlink_compact
Connections:
- H1 pad : (no net) -> standoff[0].footprint.pins[0].net-net
- H2 pad : (no net) -> standoff[1].footprint.pins[0].net-net
- J1 pad 11: jlink_interface-line-2 -> jlink_interface-line-7
- J1 pad 14: jlink_interface.idc-net-2 -> jlink_interface.idc-net
- J1 pad 15: jlink_interface-line-6 -> jlink_interface-line-2
- J1 pad 16: jlink_interface.idc-net-1 -> jlink_interface.idc-net-4
- J1 pad 17: jlink_interface-line-1 -> jlink_interface-line-3
- J1 pad 18: jlink_interface.idc-net -> jlink_interface.idc-net-3
- J1 pad 2: jlink_interface.idc-net-3 -> jlink_interface.idc-net-1
- J1 pad 20: jlink_interface.idc-net-4 -> jlink_interface.idc-net-2
- J1 pad 3: jlink_interface-line-7 -> jlink_interface-line-1
- J1 pad 5: jlink_interface-line-5 -> jlink_interface-line-6
- J1 pad 7: jlink_interface-line-3 -> jlink_interface-line-5
Changed lines of the file:
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@@
     (net 3 "jlink_interface-hv")
     (net 4 "gnd")
-    (net 5 "jlink_interface-line-1")
-    (net 6 "jlink_interface-line-6")
-    (net 7 "jlink_interface-line-2")
-    (net 8 "jlink_interface-line-3")
-    (net 9 "jlink_interface.idc-net-3")
-    (net 10 "jlink_interface-line-7")
-    (net 11 "jlink_interface-line-5")
+    (net 5 "jlink_interface-line-3")
+    (net 6 "jlink_interface-line-2")
+    (net 7 "jlink_interface-line-7")
+    (net 8 "jlink_interface-line-5")
+    (net 9 "jlink_interface.idc-net-1")
+    (net 10 "jlink_interface-line-1")
+    (net 11 "jlink_interface-line-6")
     (net 12 "jlink_interface-hv-1")
-    (net 13 "jlink_interface.idc-net")
+    (net 13 "jlink_interface.idc-net-3")
     (net 14 "jlink_interface-line-4")
-    (net 15 "jlink_interface.idc-net-2")
-    (net 16 "jlink_interface.idc-net-1")
-    (net 17 "jlink_interface.idc-net-4")
+    (net 15 "jlink_interface.idc-net")
+    (net 16 "jlink_interface.idc-net-4")
+    (net 17 "jlink_interface.idc-net-2")
     (net 18 "jlink_interface-line")
-    (footprint "atopile:CONN-SMD_20P-P2.54_BH-00019-f2b3b5"
+    (net 19 "standoff[1].footprint.pins[0].net-net")
+    (net 20 "standoff[0].footprint.pins[0].net-net")
+    (footprint "Liansheng_BH_00019:CONN-SMD_20P-P2.54_BH-00019"
         (layer "F.Cu")
         (at 0 22.5 180)
@@
         (property "Datasheet" "https://wmsc.lcsc.com/wmsc/upload/file/pdf/v2/lcsc/2105241719_Liansheng-BH-00019_C2829930.pdf"
             (at 0 0 0)
-            (layer "User.9")
-            (hide yes)
-            (effects
-                (font
-                    (size 0.125 0.125)
-                    (thickness 0.01875)
+            (layer "F.Fab")
+            (hide yes)
+            (effects
+                (font
+                    (size 1.27 1.27)
+                    (thickness 0.15)
                 )
             )
@@
             )
         )
-        (property "__atopile_lib_fp_hash__" "8f05434d-1806-86b7-eb57-456202342041"
+        (property "checksum" "c1529a46f03aaeea29e0cdcfa1d5fc2175777446f372a8cb080b83dabc8fd7cf"
+            (at 0 0 0)
+            (layer "User.9")
+            (hide yes)
+            (effects
+                (font
+                    (size 0.125 0.125)
+                    (thickness 0.01875)
+                )
+            )
+        )
+        (property "__atopile_lib_fp_hash__" "0b0583a9-1242-aa6f-3a6f-7e87aad600f2"
             (at 0 0 0)
             (layer "User.9")
@@
             (size 0.9 5)
             (layers "F.Cu" "F.Mask" "F.Paste")
-            (net 9 "jlink_interface.idc-net-3")
+            (net 9 "jlink_interface.idc-net-1")
         )
         (pad "3" smd rect
@@
             (size 0.9 5)
             (layers "F.Cu" "F.Mask" "F.Paste")
-            (net 10 "jlink_interface-line-7")
+            (net 10 "jlink_interface-line-1")
         )
         (pad "4" smd rect
@@
             (size 0.9 5)
             (layers "F.Cu" "F.Mask" "F.Paste")
-            (net 11 "jlink_interface-line-5")
+            (net 11 "jlink_interface-line-6")
         )
         (pad "6" smd rect
@@
             (size 0.9 5)
             (layers "F.Cu" "F.Mask" "F.Paste")
-            (net 8 "jlink_interface-line-3")
+            (net 8 "jlink_interface-line-5")
         )
         (pad "8" smd rect
@@
             (size 0.9 5)
             (layers "F.Cu" "F.Mask" "F.Paste")
-            (net 7 "jlink_interface-line-2")
+            (net 7 "jlink_interface-line-7")
         )
         (pad "12" smd rect
@@
             (size 0.9 5)
             (layers "F.Cu" "F.Mask" "F.Paste")
-            (net 15 "jlink_interface.idc-net-2")
+            (net 15 "jlink_interface.idc-net")
         )
         (pad "15" smd rect
@@
             (size 0.9 5)
             (layers "F.Cu" "F.Mask" "F.Paste")
-            (net 6 "jlink_interface-line-6")
+            (net 6 "jlink_interface-line-2")
         )
         (pad "16" smd rect
@@
             (size 0.9 5)
             (layers "F.Cu" "F.Mask" "F.Paste")
-            (net 16 "jlink_interface.idc-net-1")
+            (net 16 "jlink_interface.idc-net-4")
         )
         (pad "17" smd rect
@@
             (size 0.9 5)
             (layers "F.Cu" "F.Mask" "F.Paste")
-            (net 5 "jlink_interface-line-1")
+            (net 5 "jlink_interface-line-3")
         )
         (pad "18" smd rect
@@
             (size 0.9 5)
             (layers "F.Cu" "F.Mask" "F.Paste")
-            (net 13 "jlink_interface.idc-net")
+            (net 13 "jlink_interface.idc-net-3")
         )
         (pad "19" smd rect
@@
             (size 0.9 5)
             (layers "F.Cu" "F.Mask" "F.Paste")
-            (net 17 "jlink_interface.idc-net-4")
+            (net 17 "jlink_interface.idc-net-2")
         )
         (embedded_fonts no)
+        (model "${KIPRJMOD}/../../parts/Liansheng_BH_00019/CONN-SMD_20P-P2.54_BH-00019.step"
+            (offset
+                (xyz 0 0 10.5)
+            )
+            (scale
+                (xyz 1 1 1)
+            )
+            (rotate
+                (xyz 0 0 0)
+            )
+        )
     )
-    (footprint "lib:segger_jlink_compact"
+    (footprint "SEGGER_JLink_Compact:segger_jlink_compact"
         (layer "F.Cu")
         (at 0 0 0)
@@
             )
         )
-        (property "__atopile_lib_fp_hash__" "ae94fe4d-d0d8-3033-69e4-cbf5ed37651a"
+        (property "__atopile_lib_fp_hash__" "d0b66df8-1ccc-31e3-6b57-63169acaa4a1"
             (at 0 0 0)
             (layer "User.9")
@@
             (layer "F.SilkS")
         )
+        (fp_text user "${REFERENCE}"
+            (at 0 -1.6 0)
+            (layer "F.Fab")
+            (effects
+                (font
+                    (size 1 1)
+                    (thickness 0.15)
+                )
+                (hide yes)
+            )
+            (unlocked yes)
+        )
         (embedded_fonts no)
-        (model "../footprints.3dshapes/J_Link_Compact_V1.0A.step"
+        (model "${KIPRJMOD}/../../parts/SEGGER_JLink_Compact/J_Link_Compact_V1.0A.step"
             (offset
-                (xyz -16.9 -9.65 4.6)
+                (xyz -16.9 -9.65 5.6)
             )
             (scale
@@
         )
     )
-    (footprint "atopile:SMD_BD5.6-L5.6-W5.6-D4.1-1d1819"
+    (footprint "Sinhoo_SMTSO2530CTJ:SMD_BD5.6-L5.6-W5.6-D4.1"
         (layer "F.Cu")
         (at -16.1 -4.1 0)
@@
         (property "Datasheet" "https://wmsc.lcsc.com/wmsc/upload/file/pdf/v2/lcsc/2111221230_Sinhoo-SMTSO2530CTJ_C2915631.pdf"
             (at 0 0 0)
-            (layer "User.9")
-            (hide yes)
-            (effects
-                (font
-                    (size 0.125 0.125)
-                    (thickness 0.01875)
+            (layer "F.Fab")
+            (hide yes)
+            (effects
+                (font
+                    (size 1.27 1.27)
+                    (thickness 0.15)
                 )
             )
@@
             )
         )
-        (property "__atopile_lib_fp_hash__" "b6e555fa-fe21-5a8e-c85d-3361c26ec1e1"
+        (property "checksum" "80baad0f64c60e9fe2b4e2698443da69e0c68a3f1a48f47cff70c6e3a06ddf22"
+            (at 0 0 0)
+            (layer "User.9")
+            (hide yes)
+            (effects
+                (font
+                    (size 0.125 0.125)
+                    (thickness 0.01875)
+                )
+            )
+        )
+        (property "__atopile_lib_fp_hash__" "1e68b1d2-4698-05b5-c0a6-42666ba2349f"
             (at 0 0 0)
             (layer "User.9")
@@
             (drill 4.25)
             (layers "*.Cu" "*.Mask")
+            (net 19 "standoff[1].footprint.pins[0].net-net")
             (remove_unused_layers no)
         )
@@
         )
         (embedded_fonts no)
+        (model "${KIPRJMOD}/../../parts/Sinhoo_SMTSO2530CTJ/SMD_BD5.6-L5.6-W5.6-D4.1.step"
+            (offset
+                (xyz 0 0 0)
+            )
+            (scale
+                (xyz 1 1 1)
+            )
+            (rotate
+                (xyz 0 0 -90)
+            )
+        )
     )
-    (footprint "atopile:SMD_BD5.6-L5.6-W5.6-D4.1-1d1819"
+    (footprint "Sinhoo_SMTSO2530CTJ:SMD_BD5.6-L5.6-W5.6-D4.1"
         (layer "F.Cu")
         (at 16.1 -4.1 0)
@@
         (property "Datasheet" "https://wmsc.lcsc.com/wmsc/upload/file/pdf/v2/lcsc/2111221230_Sinhoo-SMTSO2530CTJ_C2915631.pdf"
             (at 0 0 0)
-            (layer "User.9")
-            (hide yes)
-            (effects
-                (font
-                    (size 0.125 0.125)
-                    (thickness 0.01875)
+            (layer "F.Fab")
+            (hide yes)
+            (effects
+                (font
+                    (size 1.27 1.27)
+                    (thickness 0.15)
                 )
             )
@@
             )
         )
-        (property "__atopile_lib_fp_hash__" "b535f677-71c1-bab5-af90-09178ab91c84"
+        (property "checksum" "80baad0f64c60e9fe2b4e2698443da69e0c68a3f1a48f47cff70c6e3a06ddf22"
+            (at 0 0 0)
+            (layer "User.9")
+            (hide yes)
+            (effects
+                (font
+                    (size 0.125 0.125)
+                    (thickness 0.01875)
+                )
+            )
+        )
+        (property "__atopile_lib_fp_hash__" "1e68b1d2-4698-05b5-c0a6-42666ba2349f"
             (at 0 0 0)
             (layer "User.9")
@@
             (drill 4.25)
             (layers "*.Cu" "*.Mask")
+            (net 20 "standoff[0].footprint.pins[0].net-net")
             (remove_unused_layers no)
         )
@@
         )
         (embedded_fonts no)
+        (model "${KIPRJMOD}/../../parts/Sinhoo_SMTSO2530CTJ/SMD_BD5.6-L5.6-W5.6-D4.1.step"
+            (offset
+                (xyz 0 0 0)
+            )
+            (scale
+                (xyz 1 1 1)
+            )
+            (rotate
+                (xyz 0 0 -90)
+            )
+        )
     )
     (embedded_fonts no)

Commit message: Manually fix fp lib tables
fix some small bugs
fix package only modules (e.g. logos)
Parts:
- MOD1: footprint SEGGER_JLink_Compact:segger_jlink_compact -> SEGGER_JLink_Compact:SEGGER_JLink_Compact
Connections:
- J1 pad 1: jlink_interface-hv-1 -> jlink_interface-hv
- J1 pad 13: jlink_interface-line-4 -> jlink_interface-line-2
- J1 pad 14: jlink_interface.idc-net -> jlink_interface.idc-net-1
- J1 pad 15: jlink_interface-line-2 -> jlink_interface-line
- J1 pad 16: jlink_interface.idc-net-4 -> jlink_interface.idc-net-3
- J1 pad 17: jlink_interface-line-3 -> jlink_interface-line-5
- J1 pad 18: jlink_interface.idc-net-3 -> jlink_interface.idc-net-4
- J1 pad 19: jlink_interface-hv -> jlink_interface-hv-1
- J1 pad 2: jlink_interface.idc-net-1 -> jlink_interface.idc-net
- J1 pad 3: jlink_interface-line-1 -> jlink_interface-line-4
- J1 pad 5: jlink_interface-line-6 -> jlink_interface-line-3
- J1 pad 7: jlink_interface-line-5 -> jlink_interface-line-1
- J1 pad 9: jlink_interface-line -> jlink_interface-line-6
Changed lines of the file:
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@@
     (net 1 "standoff[1]-contact")
     (net 2 "standoff[0]-contact")
-    (net 3 "jlink_interface-hv")
+    (net 3 "jlink_interface-hv-1")
     (net 4 "gnd")
-    (net 5 "jlink_interface-line-3")
-    (net 6 "jlink_interface-line-2")
+    (net 5 "jlink_interface-line-5")
+    (net 6 "jlink_interface-line")
     (net 7 "jlink_interface-line-7")
-    (net 8 "jlink_interface-line-5")
-    (net 9 "jlink_interface.idc-net-1")
-    (net 10 "jlink_interface-line-1")
-    (net 11 "jlink_interface-line-6")
-    (net 12 "jlink_interface-hv-1")
-    (net 13 "jlink_interface.idc-net-3")
-    (net 14 "jlink_interface-line-4")
-    (net 15 "jlink_interface.idc-net")
-    (net 16 "jlink_interface.idc-net-4")
+    (net 8 "jlink_interface-line-1")
+    (net 9 "jlink_interface.idc-net")
+    (net 10 "jlink_interface-line-4")
+    (net 11 "jlink_interface-line-3")
+    (net 12 "jlink_interface-hv")
+    (net 13 "jlink_interface.idc-net-4")
+    (net 14 "jlink_interface-line-2")
+    (net 15 "jlink_interface.idc-net-1")
+    (net 16 "jlink_interface.idc-net-3")
     (net 17 "jlink_interface.idc-net-2")
-    (net 18 "jlink_interface-line")
+    (net 18 "jlink_interface-line-6")
     (net 19 "standoff[1].footprint.pins[0].net-net")
     (net 20 "standoff[0].footprint.pins[0].net-net")
@@
             (size 0.9 5)
             (layers "F.Cu" "F.Mask" "F.Paste")
-            (net 12 "jlink_interface-hv-1")
+            (net 12 "jlink_interface-hv")
         )
         (pad "2" smd rect
@@
             (size 0.9 5)
             (layers "F.Cu" "F.Mask" "F.Paste")
-            (net 9 "jlink_interface.idc-net-1")
+            (net 9 "jlink_interface.idc-net")
         )
         (pad "3" smd rect
@@
             (size 0.9 5)
             (layers "F.Cu" "F.Mask" "F.Paste")
-            (net 10 "jlink_interface-line-1")
+            (net 10 "jlink_interface-line-4")
         )
         (pad "4" smd rect
@@
             (size 0.9 5)
             (layers "F.Cu" "F.Mask" "F.Paste")
-            (net 11 "jlink_interface-line-6")
+            (net 11 "jlink_interface-line-3")
         )
         (pad "6" smd rect
@@
             (size 0.9 5)
             (layers "F.Cu" "F.Mask" "F.Paste")
-            (net 8 "jlink_interface-line-5")
+            (net 8 "jlink_interface-line-1")
         )
         (pad "8" smd rect
@@
             (size 0.9 5)
             (layers "F.Cu" "F.Mask" "F.Paste")
-            (net 18 "jlink_interface-line")
+            (net 18 "jlink_interface-line-6")
         )
         (pad "10" smd rect
@@
             (size 0.9 5)
             (layers "F.Cu" "F.Mask" "F.Paste")
-            (net 14 "jlink_interface-line-4")
+            (net 14 "jlink_interface-line-2")
         )
         (pad "14" smd rect
@@
             (size 0.9 5)
             (layers "F.Cu" "F.Mask" "F.Paste")
-            (net 15 "jlink_interface.idc-net")
+            (net 15 "jlink_interface.idc-net-1")
         )
         (pad "15" smd rect
@@
             (size 0.9 5)
             (layers "F.Cu" "F.Mask" "F.Paste")
-            (net 6 "jlink_interface-line-2")
+            (net 6 "jlink_interface-line")
         )
         (pad "16" smd rect
@@
             (size 0.9 5)
             (layers "F.Cu" "F.Mask" "F.Paste")
-            (net 16 "jlink_interface.idc-net-4")
+            (net 16 "jlink_interface.idc-net-3")
         )
         (pad "17" smd rect
@@
             (size 0.9 5)
             (layers "F.Cu" "F.Mask" "F.Paste")
-            (net 5 "jlink_interface-line-3")
+            (net 5 "jlink_interface-line-5")
         )
         (pad "18" smd rect
@@
             (size 0.9 5)
             (layers "F.Cu" "F.Mask" "F.Paste")
-            (net 13 "jlink_interface.idc-net-3")
+            (net 13 "jlink_interface.idc-net-4")
         )
         (pad "19" smd rect
@@
             (size 0.9 5)
             (layers "F.Cu" "F.Mask" "F.Paste")
-            (net 3 "jlink_interface-hv")
+            (net 3 "jlink_interface-hv-1")
         )
         (pad "20" smd rect
@@
         )
     )
-    (footprint "SEGGER_JLink_Compact:segger_jlink_compact"
+    (footprint "SEGGER_JLink_Compact:SEGGER_JLink_Compact"
         (layer "F.Cu")
         (at 0 0 0)
@@
             )
         )
-        (property "__atopile_lib_fp_hash__" "d0b66df8-1ccc-31e3-6b57-63169acaa4a1"
-            (at 0 0 0)
-            (layer "User.9")
+        (property "__atopile_lib_fp_hash__" "67822b65-6f55-9d9c-817a-545e30d0c574"
+            (at 0 0 0)
+            (layer "User.9")

Commit message: rebuild all packages & regenerate images of changed layouts (silk)
Add new scripts for version bump and build (based on atopile/packages)
Connections:
- net jlink_interface.idc-net renamed _2
- net jlink_interface.idc-net-1 renamed _14
- net jlink_interface.idc-net-2 renamed _20
- net jlink_interface.idc-net-3 renamed _16
- net jlink_interface.idc-net-4 renamed _18
- J1 pad 11: jlink_interface-line-7 -> jlink_interface-line
- J1 pad 13: jlink_interface-line-2 -> jlink_interface-line-1
- J1 pad 15: jlink_interface-line -> jlink_interface-line-2
- J1 pad 17: jlink_interface-line-5 -> jlink_interface-line-3
- J1 pad 5: jlink_interface-line-3 -> jlink_interface-line-5
- J1 pad 7: jlink_interface-line-1 -> jlink_interface-line-6
- J1 pad 9: jlink_interface-line-6 -> jlink_interface-line-7
