File: packages/analog-devices-max14778/layouts/analog_devices_max14778_driver/analog_devices_max14778_driver.kicad_pcb (KiCad board)
At the start: 2 copper layers, 4 parts

Commit message: Update analog_devices_max14778
Parts:
- C1: footprint atopile:C0402-b3ef17 -> Samsung_Electro_Mechanics_CL05B104KO5NNNC:C0402
- C2, C3: footprint atopile:C0603-bd72f6 -> FH_0603B104K101NT:C0603
- U1: footprint atopile:TQFN-20_L5.0-W5.0-P0.65-TL-EP3.1-c7465b -> Maxim_Integrated_MAX14778ETP_T:TQFN-20_L5.0-W5.0-P0.65-TL-EP3.1
Connections:
- net EP renamed VN

Commit message: WIP update packages till ESPs
Connections:
- net VN renamed EP

Commit message: Manually fix fp lib tables
fix some small bugs
fix package only modules (e.g. logos)
Connections:
- net EP renamed VN

Commit message: rebuild all packages & regenerate images of changed layouts (silk)
Add new scripts for version bump and build (based on atopile/packages)
Connections:
- net VN renamed EP
Changed lines of the file:
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@@
     (net 0 "")
     (net 1 "output_a[2]")
-    (net 2 "VN")
+    (net 2 "EP")
     (net 3 "common_a")
     (net 4 "SA0")
@@
             (size 0.8 0.9)
             (layers "F.Cu" "F.Mask" "F.Paste")
-            (net 2 "VN")
+            (net 2 "EP")
         )
         (pad "2" smd rect
@@
             (size 0.4 0.95)
             (layers "F.Cu" "F.Mask" "F.Paste")
-            (net 2 "VN")
+            (net 2 "EP")
         )
         (pad "5" smd rect
@@
             (size 3.1 3.1)
             (layers "F.Cu" "F.Mask" "F.Paste")
-            (net 2 "VN")
+            (net 2 "EP")
         )
         (embedded_fonts no)

Commit message: Use packages from packages folder
Parts:
- C2, C3: footprint FH_0603B104K101NT:C0603 -> YAGEO_CC0603KRX7R0BB104:C0603
