File: packages/leds/layouts/addressable_led_connector_driver/addressable_led_connector_driver.kicad_pcb (KiCad board)
At the start: 2 copper layers, 1 part

Commit message: rebuild all packages & regenerate images of changed layouts (silk)
Add new scripts for version bump and build (based on atopile/packages)
Connections:
- U1 pad 3: line-1 -> line
- U1 pad 4: line -> line-1
Changed lines of the file:
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@@
     )
     (net 0 "")
-    (net 1 "line-1")
+    (net 1 "line")
     (net 2 "gnd")
-    (net 3 "line")
+    (net 3 "line-1")
     (net 4 "hv")
     (footprint "Changzhou_Amass_Elec_XT30PW_2_2__M_G_B:CONN-TH_4P-XT30PW-M"
@@
             (drill 0.9144)
             (layers "*.Cu" "*.Mask")
-            (net 1 "line-1")
+            (net 1 "line")
             (remove_unused_layers no)
         )
@@
             (drill 0.9144)
             (layers "*.Cu" "*.Mask")
-            (net 3 "line")
+            (net 3 "line-1")
             (remove_unused_layers no)
         )

Commit message: Use packages from packages folder
Connections:
- U1 pad 3: line -> line-1
- U1 pad 4: line-1 -> line
