File: packages/rs485/layouts/analog_devices_adm2587ebrwz_driver/analog_devices_adm2587ebrwz_driver.kicad_pcb (KiCad board)
At the start: 2 copper layers, 9 parts

Commit message: WIP update rs485
Parts:
- C1, C3, C5, C7: footprint atopile:C0603-bd72f6 -> YAGEO_CC0603JRX7R9BB104:C0603
- C2, C4, C6, C8: footprint atopile:C0603-bd72f6 -> FH_0603B103J500NT:C0603
- U1: footprint atopile:SOIC-20_L13.0-W7.6-P1.27-LS10.3-BL-5ed090 -> Analog_Devices_ADM2587EBRWZ_REEL7:SOIC-20_L13.0-W7.6-P1.27-LS10.3-BL
Connections:
- C1 pad 1: hv -> hv-1
- C2 pad 1: hv -> hv-1
- C3 pad 1: hv -> hv-1
- C4 pad 1: hv -> hv-1
- C5 pad 1: hv-1 -> hv
- C6 pad 1: hv-1 -> hv
- C7 pad 1: hv-1 -> hv
- C8 pad 1: hv-1 -> hv
- U1 pad 12: hv -> hv-1
- U1 pad 13: line -> line-4
- U1 pad 15: line-2 -> line-3
- U1 pad 17: line-2 -> line-3
- U1 pad 18: line -> line-4
- U1 pad 19: hv -> hv-1
- U1 pad 2: hv-1 -> hv
- U1 pad 4: line-4 -> line
- U1 pad 5: line-3 -> line-2
- U1 pad 6: line-3 -> line-2
- U1 pad 8: hv-1 -> hv
Routing:
- net line-4: track 0.00 -> 13.8 mm, vias 0 -> 1
- net line: track 13.8 -> 0.00 mm, vias 1 -> 0
- net hv-1: track 8.09 -> 16.9 mm
- net hv: track 16.9 -> 8.09 mm
- net line-3: track 4.35 -> 9.87 mm, vias 0 -> 1
- net line-2: track 9.87 -> 4.35 mm, vias 1 -> 0

Commit message: Manually fix fp lib tables
fix some small bugs
fix package only modules (e.g. logos)
Connections:
- U1 pad 13: line-4 -> line
- U1 pad 15: line-3 -> line-4
- U1 pad 17: line-3 -> line-4
- U1 pad 18: line-4 -> line
- U1 pad 4: line -> line-3
Routing:
- net line: track 0.00 -> 13.8 mm, vias 0 -> 1
- net line-3: track 9.87 -> 0.00 mm, vias 1 -> 0
- net line-4: track 13.8 -> 9.87 mm
Changed lines of the file:
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@@
     (net 0 "")
     (net 1 "hv-1")
-    (net 2 "line")
+    (net 2 "line-3")
     (net 3 "gnd")
-    (net 4 "line-4")
+    (net 4 "line")
     (net 5 "hv")
-    (net 6 "line-3")
+    (net 6 "line-4")
     (net 7 "line-1")
     (net 8 "gnd-1")
@@
             )
         )
-        (property "__atopile_lib_fp_hash__" "dcb0a25b-9084-4c5e-0c80-abb49503373e"
+        (property "__atopile_lib_fp_hash__" "d4db9b1a-b023-62c4-2f0a-1ccb35300f69"
             (at 0 0 0)
             (layer "User.9")
@@
             )
         )
-        (property "checksum" "a4bed73005cdefa8138f25e93aae25104dd152614e8e775ce38410abab0748ed"
+        (property "checksum" "09926d95dcd81b52ff433ee1cec95741403b7e18063d143f33754534b0fc1205"
             (at 0 0 0)
             (layer "User.9")
@@
             (net 5 "hv")
         )
-        (model "${KIPRJMOD}/../../build/cache/parts/easyeda/C91183/C0603_L1.6-W0.8-H0.8.step"
+        (model "${KIPRJMOD}/../../parts/YAGEO_CC0603JRX7R9BB104/C0603_L1.6-W0.8-H0.8.step"
             (offset
                 (xyz 0 0 0)
@@
             )
         )
-        (property "__atopile_lib_fp_hash__" "0f7fac94-75de-bc4f-e9b1-6960d0f35a65"
+        (property "__atopile_lib_fp_hash__" "e4a0c806-c781-634e-43d7-d63816f5c4b4"
             (at 0 0 0)
             (layer "User.9")
@@
             )
         )
-        (property "checksum" "2cbeb4b9d1085d31910c1e066310749a40a41dcdde753b5d563fa8985e91ff77"
+        (property "checksum" "75d3d7da978a8ebe09358726f781e979cb201ccac6a2ec660ff5b2dfc3021bec"
             (at 0 0 0)
             (layer "User.9")
@@
             (net 5 "hv")
         )
-        (model "${KIPRJMOD}/../../build/cache/parts/easyeda/C124567/C0603_L1.6-W0.8-H0.8.step"
+        (model "${KIPRJMOD}/../../parts/FH_0603B103J500NT/C0603_L1.6-W0.8-H0.8.step"
             (offset
                 (xyz 0 0 0)
@@
             )
         )
-        (property "__atopile_lib_fp_hash__" "dcb0a25b-9084-4c5e-0c80-abb49503373e"
+        (property "__atopile_lib_fp_hash__" "d4db9b1a-b023-62c4-2f0a-1ccb35300f69"
             (at 0 0 0)
             (layer "User.9")
@@
             )
         )
-        (property "checksum" "a4bed73005cdefa8138f25e93aae25104dd152614e8e775ce38410abab0748ed"
+        (property "checksum" "09926d95dcd81b52ff433ee1cec95741403b7e18063d143f33754534b0fc1205"
             (at 0 0 0)
             (layer "User.9")
@@
             (net 1 "hv-1")
         )
-        (model "${KIPRJMOD}/../../build/cache/parts/easyeda/C91183/C0603_L1.6-W0.8-H0.8.step"
+        (model "${KIPRJMOD}/../../parts/YAGEO_CC0603JRX7R9BB104/C0603_L1.6-W0.8-H0.8.step"
             (offset
                 (xyz 0 0 0)
@@
             )
         )
-        (property "__atopile_lib_fp_hash__" "dcb0a25b-9084-4c5e-0c80-abb49503373e"
+        (property "__atopile_lib_fp_hash__" "d4db9b1a-b023-62c4-2f0a-1ccb35300f69"
             (at 0 0 0)
             (layer "User.9")
@@
             )
         )
-        (property "checksum" "a4bed73005cdefa8138f25e93aae25104dd152614e8e775ce38410abab0748ed"
+        (property "checksum" "09926d95dcd81b52ff433ee1cec95741403b7e18063d143f33754534b0fc1205"
             (at 0 0 0)
             (layer "User.9")
@@
             (net 5 "hv")
         )
-        (model "${KIPRJMOD}/../../build/cache/parts/easyeda/C91183/C0603_L1.6-W0.8-H0.8.step"
+        (model "${KIPRJMOD}/../../parts/YAGEO_CC0603JRX7R9BB104/C0603_L1.6-W0.8-H0.8.step"
             (offset
                 (xyz 0 0 0)
@@
             )
         )
-        (property "__atopile_lib_fp_hash__" "dcb0a25b-9084-4c5e-0c80-abb49503373e"
+        (property "__atopile_lib_fp_hash__" "d4db9b1a-b023-62c4-2f0a-1ccb35300f69"
             (at 0 0 0)
             (layer "User.9")
@@
             )
         )
-        (property "checksum" "a4bed73005cdefa8138f25e93aae25104dd152614e8e775ce38410abab0748ed"
+        (property "checksum" "09926d95dcd81b52ff433ee1cec95741403b7e18063d143f33754534b0fc1205"
             (at 0 0 0)
             (layer "User.9")
@@
             (net 1 "hv-1")
         )
-        (model "${KIPRJMOD}/../../build/cache/parts/easyeda/C91183/C0603_L1.6-W0.8-H0.8.step"
+        (model "${KIPRJMOD}/../../parts/YAGEO_CC0603JRX7R9BB104/C0603_L1.6-W0.8-H0.8.step"
             (offset
                 (xyz 0 0 0)
@@
             )
         )
-        (property "__atopile_lib_fp_hash__" "0f7fac94-75de-bc4f-e9b1-6960d0f35a65"
+        (property "__atopile_lib_fp_hash__" "e4a0c806-c781-634e-43d7-d63816f5c4b4"
             (at 0 0 0)
             (layer "User.9")
@@
             )
         )
-        (property "checksum" "2cbeb4b9d1085d31910c1e066310749a40a41dcdde753b5d563fa8985e91ff77"
+        (property "checksum" "75d3d7da978a8ebe09358726f781e979cb201ccac6a2ec660ff5b2dfc3021bec"
             (at 0 0 0)
             (layer "User.9")
@@
             (net 1 "hv-1")
         )
-        (model "${KIPRJMOD}/../../build/cache/parts/easyeda/C124567/C0603_L1.6-W0.8-H0.8.step"
+        (model "${KIPRJMOD}/../../parts/FH_0603B103J500NT/C0603_L1.6-W0.8-H0.8.step"
             (offset
                 (xyz 0 0 0)
@@
             )
         )
-        (property "__atopile_lib_fp_hash__" "9bfe8dee-6c40-0784-2a89-b413ebf95210"
+        (property "__atopile_lib_fp_hash__" "dfcae175-f3e9-cf5c-3be3-1b093945f8c6"
             (at 0 0 0)
             (layer "User.9")
@@
             )
         )
-        (property "checksum" "1453503dbf0fc79efbcc9f655fa7b999a66799053961e8f57d6218290a1f3bb4"
+        (property "checksum" "be95d8f45d9bd2bae067b28a190f91aaa07029972d69693c5919eb3e7c6e63d2"
             (at 0 0 0)
             (layer "User.9")
@@
             (size 0.59 2.36)
             (layers "F.Cu" "F.Paste" "F.Mask")
-            (net 2 "line")
+            (net 2 "line-3")
         )
         (pad "5" smd oval
@@
             (size 0.59 2.36)
             (layers "F.Cu" "F.Paste" "F.Mask")
-            (net 4 "line-4")
+            (net 4 "line")
         )
         (pad "17" smd oval
@@
             (size 0.59 2.36)
             (layers "F.Cu" "F.Paste" "F.Mask")
-            (net 6 "line-3")
+            (net 6 "line-4")
         )
         (pad "16" smd oval
@@
             (size 0.59 2.36)
             (layers "F.Cu" "F.Paste" "F.Mask")
-            (net 6 "line-3")
+            (net 6 "line-4")
         )
         (pad "14" smd oval
@@
             (size 0.59 2.36)
             (layers "F.Cu" "F.Paste" "F.Mask")
-            (net 4 "line-4")
+            (net 4 "line")
         )
         (pad "12" smd oval
@@
             (net 3 "gnd")
         )
-        (model "${KIPRJMOD}/../../build/cache/parts/easyeda/C12081/SOIC-20_L12.8-W7.5-H2.7-LS10.3-P1.27.step"
+        (model "${KIPRJMOD}/../../parts/Analog_Devices_ADM2587EBRWZ_REEL7/SOIC-20_L12.8-W7.5-H2.7-LS10.3-P1.27.step"
             (offset
                 (xyz 0 0 0)
@@
             )
         )
-        (property "__atopile_lib_fp_hash__" "0f7fac94-75de-bc4f-e9b1-6960d0f35a65"
+        (property "__atopile_lib_fp_hash__" "e4a0c806-c781-634e-43d7-d63816f5c4b4"
             (at 0 0 0)
             (layer "User.9")
@@
             )
         )
-        (property "checksum" "2cbeb4b9d1085d31910c1e066310749a40a41dcdde753b5d563fa8985e91ff77"
+        (property "checksum" "75d3d7da978a8ebe09358726f781e979cb201ccac6a2ec660ff5b2dfc3021bec"
             (at 0 0 0)
             (layer "User.9")
@@
             (net 1 "hv-1")
         )
-        (model "${KIPRJMOD}/../../build/cache/parts/easyeda/C124567/C0603_L1.6-W0.8-H0.8.step"
+        (model "${KIPRJMOD}/../../parts/FH_0603B103J500NT/C0603_L1.6-W0.8-H0.8.step"
             (offset
                 (xyz 0 0 0)
@@
             )
         )
-        (property "__atopile_lib_fp_hash__" "0f7fac94-75de-bc4f-e9b1-6960d0f35a65"
+        (property "__atopile_lib_fp_hash__" "e4a0c806-c781-634e-43d7-d63816f5c4b4"
             (at 0 0 0)
             (layer "User.9")
@@
             )
         )
-        (property "checksum" "2cbeb4b9d1085d31910c1e066310749a40a41dcdde753b5d563fa8985e91ff77"
+        (property "checksum" "75d3d7da978a8ebe09358726f781e979cb201ccac6a2ec660ff5b2dfc3021bec"
             (at 0 0 0)
             (layer "User.9")
@@
             (net 5 "hv")
         )
-        (model "${KIPRJMOD}/../../build/cache/parts/easyeda/C124567/C0603_L1.6-W0.8-H0.8.step"
+        (model "${KIPRJMOD}/../../parts/FH_0603B103J500NT/C0603_L1.6-W0.8-H0.8.step"
             (offset
                 (xyz 0 0 0)

Commit message: Update 3D model locations
fix missing renders
Connections:
- U1 pad 13: line -> line-3
- U1 pad 15: line-4 -> line-1
- U1 pad 17: line-4 -> line-1
- U1 pad 18: line -> line-3
- U1 pad 4: line-3 -> line-4
- U1 pad 7: line-1 -> line
Routing:
- net line-3: track 0.00 -> 13.8 mm, vias 0 -> 1
- net line: track 13.8 -> 0.00 mm, vias 1 -> 0
- net line-4: track 9.87 -> 0.00 mm, vias 1 -> 0
- net line-1: track 0.00 -> 9.87 mm, vias 0 -> 1

Commit message: rebuild all packages & regenerate images of changed layouts (silk)
Add new scripts for version bump and build (based on atopile/packages)
Connections:
- C1 pad 1: hv-1 -> hv
- C2 pad 1: hv-1 -> hv
- C3 pad 1: hv-1 -> hv
- C4 pad 1: hv-1 -> hv
- C5 pad 1: hv -> hv-1
- C6 pad 1: hv -> hv-1
- C7 pad 1: hv -> hv-1
- C8 pad 1: hv -> hv-1
- U1 pad 12: hv-1 -> hv
- U1 pad 13: line-3 -> line-2
- U1 pad 18: line-3 -> line-2
- U1 pad 19: hv-1 -> hv
- U1 pad 2: hv -> hv-1
- U1 pad 4: line-4 -> line-3
- U1 pad 5: line-2 -> line
- U1 pad 6: line-2 -> line
- U1 pad 7: line -> line-4
- U1 pad 8: hv -> hv-1
Routing:
- net line-3: track 13.8 -> 0.00 mm, vias 1 -> 0
- net line-2: track 4.35 -> 13.8 mm, vias 0 -> 1
- net hv-1: track 16.9 -> 8.09 mm
- net hv: track 8.09 -> 16.9 mm
- net line: track 0.00 -> 4.35 mm
Changed lines of the file:
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@@
     )
     (net 0 "")
-    (net 1 "hv-1")
-    (net 2 "line-4")
+    (net 1 "hv")
+    (net 2 "line-3")
     (net 3 "gnd")
-    (net 4 "line-3")
-    (net 5 "hv")
+    (net 4 "line-2")
+    (net 5 "hv-1")
     (net 6 "line-1")
-    (net 7 "line")
+    (net 7 "line-4")
     (net 8 "gnd-1")
-    (net 9 "line-2")
+    (net 9 "line")
     (footprint "YAGEO_CC0603JRX7R9BB104:C0603"
         (layer "F.Cu")
@@
             (size 0.8 0.9)
             (layers "F.Cu" "F.Mask" "F.Paste")
-            (net 5 "hv")
+            (net 5 "hv-1")
         )
         (pad "2" smd rect
@@
             (size 0.8 0.9)
             (layers "F.Cu" "F.Mask" "F.Paste")
-            (net 5 "hv")
+            (net 5 "hv-1")
         )
         (pad "2" smd rect
@@
             (size 0.8 0.9)
             (layers "F.Cu" "F.Mask" "F.Paste")
-            (net 1 "hv-1")
+            (net 1 "hv")
         )
         (pad "2" smd rect
@@
             (size 0.8 0.9)
             (layers "F.Cu" "F.Mask" "F.Paste")
-            (net 5 "hv")
+            (net 5 "hv-1")
         )
         (pad "2" smd rect
@@
             (size 0.8 0.9)
             (layers "F.Cu" "F.Mask" "F.Paste")
-            (net 1 "hv-1")
+            (net 1 "hv")
         )
         (pad "2" smd rect
@@
             (size 0.8 0.9)
             (layers "F.Cu" "F.Mask" "F.Paste")
-            (net 1 "hv-1")
+            (net 1 "hv")
         )
         (pad "2" smd rect
@@
             (size 0.59 2.36)
             (layers "F.Cu" "F.Mask" "F.Paste")
-            (net 5 "hv")
+            (net 5 "hv-1")
         )
         (pad "3" smd oval
@@
             (size 0.59 2.36)
             (layers "F.Cu" "F.Mask" "F.Paste")
-            (net 2 "line-4")
+            (net 2 "line-3")
         )
         (pad "5" smd oval
@@
             (size 0.59 2.36)
             (layers "F.Cu" "F.Mask" "F.Paste")
-            (net 9 "line-2")
+            (net 9 "line")
         )
         (pad "6" smd oval
@@
             (size 0.59 2.36)
             (layers "F.Cu" "F.Mask" "F.Paste")
-            (net 9 "line-2")
+            (net 9 "line")
         )
         (pad "7" smd oval
@@
             (size 0.59 2.36)
             (layers "F.Cu" "F.Mask" "F.Paste")
-            (net 7 "line")
+            (net 7 "line-4")
         )
         (pad "8" smd oval
@@
             (size 0.59 2.36)
             (layers "F.Cu" "F.Mask" "F.Paste")
-            (net 5 "hv")
+            (net 5 "hv-1")
         )
         (pad "9" smd oval
@@
             (size 0.59 2.36)
             (layers "F.Cu" "F.Mask" "F.Paste")
-            (net 1 "hv-1")
+            (net 1 "hv")
         )
         (pad "13" smd oval
@@
             (size 0.59 2.36)
             (layers "F.Cu" "F.Mask" "F.Paste")
-            (net 4 "line-3")
+            (net 4 "line-2")
         )
         (pad "14" smd oval
@@
             (size 0.59 2.36)
             (layers "F.Cu" "F.Mask" "F.Paste")
-            (net 4 "line-3")
+            (net 4 "line-2")
         )
         (pad "19" smd oval
@@
             (size 0.59 2.36)
             (layers "F.Cu" "F.Mask" "F.Paste")
-            (net 1 "hv-1")
+            (net 1 "hv")
         )
         (pad "20" smd oval
@@
             (size 0.8 0.9)
             (layers "F.Cu" "F.Mask" "F.Paste")
-            (net 1 "hv-1")
+            (net 1 "hv")
         )
         (pad "2" smd rect
@@
             (size 0.8 0.9)
             (layers "F.Cu" "F.Mask" "F.Paste")
-            (net 5 "hv")
+            (net 5 "hv-1")
         )
         (pad "2" smd rect
